File: KiCad/Bell2.kicad_pcb (KiCad board)
At the start: 2 copper layers, 34.8 x 27.5 mm, 34 parts, among them J1 USB-C, J2 POWER, J3 Conn_01x10, U1 ESP32-PICO-MINI-02, U2 FT231XQ, U3 ISL89410, U4 ISL89410, U5 LMR16006+FB, U6 AA, U7 QR

Commit message: Started Keypad2 - may scrap it though.
Parts:
- R10: value 324R -> 220R
- R8: value 732R -> 680R
Changed lines of the file:
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@@
       (effects (font (size 0.5 0.5) (thickness 0.08)))
     )
-    (fp_text value "324R" (at 0 0) (layer "F.Fab")
+    (fp_text value "220R" (at 0 0) (layer "F.Fab")
       (effects (font (size 0.4 0.4) (thickness 0.08)))
     )
@@
       (effects (font (size 0.5 0.5) (thickness 0.08)))
     )
-    (fp_text value "732R" (at 0 0) (layer "F.Fab")
-      (effects (font (size 0.4 0.4) (thickness 0.08)))
-    )
+    (fp_text value "680R" (at 0 0) (layer "F.Fab")
+      (effects (font (size 0.4 0.4) (thickness 0.08)))
+    )

Commit message: Bell2 - tracks and DRC
Parts:
- C2, C3: moved to B.Cu
- moved AJK1 56.3 mm to (104.5, 50.5)
- moved U6 48.9 mm to (105.2, 57.8)
- moved C3 37.5 mm to (105.0, 43.0)
- moved C2 34.8 mm to (105.0, 38.0), turned to 180 degrees
- moved R7 30.9 mm to (99.3, 39.8), turned to 90 degrees
- moved R4 29.1 mm to (99.3, 37.1), turned to -90 degrees
- moved R11 28.3 mm to (74.0, 58.8), turned to 90 degrees
- moved U7 28.1 mm to (80.0, 44.2), turned to 0 degrees
- moved R3 24.9 mm to (91.2, 50.8)
- moved R10 24.1 mm to (89.0, 42.8), turned to 180 degrees
- moved R5 23.7 mm to (85.0, 52.2), turned to 180 degrees
- moved C1 23.0 mm to (93.2, 34.0), turned to 180 degrees
- moved R2 22.4 mm to (91.3, 49.2)
- moved R9 20.9 mm to (89.0, 41.5), turned to 180 degrees
- moved R6 20.3 mm to (90.2, 52.2), turned to 180 degrees
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Connections:
- U1 pad 12: R -> unconnected-(U1-Pad12)
- U1 pad 13: G -> unconnected-(U1-Pad13)
- U1 pad 15: OUT3 -> unconnected-(U1-Pad15)
- U1 pad 16: OUT4 -> unconnected-(U1-Pad16)
- U1 pad 17: B -> unconnected-(U1-Pad17)
- U1 pad 18: unconnected-(U1-Pad18) -> OUT1
- U1 pad 20: unconnected-(U1-Pad20) -> OUT2
- U1 pad 21: unconnected-(U1-Pad21) -> OUT3
- U1 pad 27: unconnected-(U1-Pad27) -> IN1
- U1 pad 28: unconnected-(U1-Pad28) -> OUT4
- U1 pad 33: IN1 -> R
- U1 pad 34: OUT2 -> B
- U1 pad 35: OUT1 -> G
Routing:
- net +3V3: track 0.00 -> 85.1 mm, vias 0 -> 6
- net +12V: track 0.00 -> 50.1 mm, vias 0 -> 4
- net EN: track 0.00 -> 43.7 mm, vias 0 -> 3
- net GND: track 0.00 -> 37.7 mm, vias 0 -> 6
- net IN1: track 0.00 -> 30.2 mm, vias 0 -> 2
- net D+: track 0.00 -> 29.6 mm, vias 0 -> 3
- net IN2: track 0.00 -> 28.9 mm, vias 0 -> 2
- net BOOT: track 0.00 -> 26.3 mm, vias 0 -> 2
- net OUT1: track 0.00 -> 25.0 mm, vias 0 -> 2
- net D-: track 0.00 -> 24.9 mm, vias 0 -> 3
- net OUT3: track 0.00 -> 23.4 mm, vias 0 -> 2
- net OUT2: track 0.00 -> 21.8 mm, vias 0 -> 2
- net I: track 0.00 -> 21.4 mm, vias 0 -> 2
- net Net-(R2-Pad2): track 0.00 -> 20.6 mm
- net VBUS: track 0.00 -> 16.9 mm
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- added copper zone on B.Cu, net GND
- added copper zone on F.Cu, net GND
Other:
- board text added: "www.me.uk"

Commit message: Checking
Parts:
- U2: footprint RevK:QFN-20-1EP_4x4mm_P0.5mm_EP2.5x2.5mm -> Package_DFN_QFN:QFN-20-1EP_4x4mm_P0.5mm_EP2.5x2.5mm
Routing:
- net GND: track 37.7 -> 40.9 mm
- net IN2: track 28.9 -> 26.9 mm
- net OUT2: track 21.8 -> 20.3 mm
- net OUT1: track 25.0 -> 23.6 mm
- net +12V: track 50.1 -> 48.8 mm
- net D+: track 29.6 -> 28.4 mm
- net D-: track 24.9 -> 23.9 mm
- net +3V3: track 85.1 -> 85.8 mm
- net B: track 3.26 -> 3.81 mm
- net OUT3: track 23.4 -> 22.9 mm
- net BOOT: track 26.3 -> 25.8 mm

Commit message: Tidy
Parts:
- moved C5 43.6 mm to (81.0, 58.5)
- moved C6 42.8 mm to (81.0, 52.3)
- moved C4 39.6 mm to (77.8, 59.8)
- moved D4 30.6 mm to (80.7, 55.4), turned to 90 degrees
- moved L1 25.5 mm to (77.5, 53.8), turned to 90 degrees
Routing:
- net GND: track 40.9 -> 35.8 mm, vias 6 -> 7
- net VBUS: track 16.6 -> 18.3 mm
- net IN1: track 29.9 -> 30.4 mm
Other:
- board text added: "Solar System Bell Box"

Commit message: Tidy
Parts:
- U2: footprint Package_DFN_QFN:QFN-20-1EP_4x4mm_P0.5mm_EP2.5x2.5mm -> RevK:QFN-20-1EP_4x4mm_P0.5mm_EP2.5x2.5mm

Commit message: Tidy
Other:
- board text removed: "www.me.uk"
Changed lines of the file:
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@@
       (effects (font (size 1 1) (thickness 0.15)) (justify mirror))
     )
-    (fp_line (start 0 0) (end -1.5 0) (layer "B.Cu") (width 0.25))
-    (fp_line (start 0 0) (end 1.8 -2.1) (layer "B.Cu") (width 0.25))
+    (fp_text user "www.me.uk" (at -0.58 -3.75 unlocked) (layer "B.SilkS")
+      (effects (font (size 0.65 0.65) (thickness 0.1)) (justify mirror))
+    )
+    (fp_line (start 0 2.1) (end 0 -2.1) (layer "B.Cu") (width 0.25))
+    (fp_line (start 0 2.1) (end -3 -2.1) (layer "B.Cu") (width 0.25))
+    (fp_line (start 1.8 2) (end 0 0) (layer "B.Cu") (width 0.25))
+    (fp_line (start -0.85 -1.95) (end -0.85 -2.25) (layer "B.Cu") (width 0.08))
     (fp_line (start -0.75 -2.11) (end -0.65 -2.25) (layer "B.Cu") (width 0.08))
     (fp_line (start -0.85 -2.11) (end -0.75 -2.11) (layer "B.Cu") (width 0.08))
-    (fp_line (start -0.85 -1.95) (end -0.85 -2.25) (layer "B.Cu") (width 0.08))
-    (fp_line (start 0 2.1) (end -3 -2.1) (layer "B.Cu") (width 0.25))
-    (fp_line (start 1.8 2) (end 0 0) (layer "B.Cu") (width 0.25))
+    (fp_line (start 0 0) (end 1.8 -2.1) (layer "B.Cu") (width 0.25))
+    (fp_line (start 0 0) (end -1.5 0) (layer "B.Cu") (width 0.25))
     (fp_line (start -0.85 -1.95) (end -0.75 -1.95) (layer "B.Cu") (width 0.08))
-    (fp_line (start 0 2.1) (end 0 -2.1) (layer "B.Cu") (width 0.25))
+    (fp_arc (start -1.5 -2.1) (mid -0.75 -2.85) (end 0 -2.1) (layer "B.Cu") (width 0.25))
     (fp_arc (start -0.75 -2.11) (mid -0.67 -2.03) (end -0.75 -1.95) (layer "B.Cu") (width 0.08))
-    (fp_arc (start -1.5 -2.1) (mid -0.75 -2.85) (end 0 -2.1) (layer "B.Cu") (width 0.25))
     (fp_circle (center -0.77 -2.11) (end -0.47 -2.11) (layer "B.Cu") (width 0.08) (fill none))
+    (fp_line (start 0 2.1) (end 0 -2.1) (layer "B.Mask") (width 0.45))
     (fp_line (start 0 0) (end -1.5 0) (layer "B.Mask") (width 0.45))
-    (fp_line (start 0 2.1) (end 0 -2.1) (layer "B.Mask") (width 0.45))
-    (fp_line (start 0 2.1) (end -3 -2.1) (layer "B.Mask") (width 0.45))
     (fp_line (start 0 0) (end 1.8 -2.1) (layer "B.Mask") (width 0.45))
     (fp_line (start 1.8 2) (end 0 0) (layer "B.Mask") (width 0.45))
+    (fp_line (start 0 2.1) (end -3 -2.1) (layer "B.Mask") (width 0.45))
     (fp_arc (start -1.5 -2.1) (mid -0.75 -2.85) (end 0 -2.1) (layer "B.Mask") (width 0.45))
   )
@@
     (effects (font (size 1 1) (thickness 0.15)) (justify mirror))
   )
-  (gr_text "www.me.uk" (at 105 54.25) (layer "B.SilkS")
-    (effects (font (size 0.7 0.7) (thickness 0.1)) (justify mirror))
-  )
   (dimension (type aligned) (layer "Dwgs.User")

Commit message: Tidy
Parts:
- moved AJK1 1.38 mm to (104.4, 49.1)
- moved U6 1.38 mm to (105.2, 56.4)
- moved R6 0.25 mm to (90.0, 52.2)
- moved U7 0.11 mm to (80.1, 44.2)
Routing:
- net D+: track 28.4 -> 20.6 mm, vias 3 -> 2
- net D-: track 23.9 -> 21.1 mm, vias 3 -> 2
- net VBUS: track 18.3 -> 15.6 mm
- net +3V3: track 85.7 -> 87.8 mm
- net OUT1: track 23.6 -> 21.9 mm
- net IN1: track 30.4 -> 31.8 mm
- net GND: track 35.8 -> 35.7 mm, vias 7 -> 8
Other:
- board text added: "12V"
- board text added: "BELL"
- board text added: "BKLT"
- board text added: "ENG"
- board text added: "FAULT"
- board text added: "GND"
- board text added: "STB"
- board text added: "TAMPER"

Commit message: Silkscreen
Other:
- board text added: "Solar System Bell2"
- board text removed: "Solar System Bell Box"
Changed lines of the file:
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@@
   (gr_line (start 73.25 38.5) (end 91.5 38.5) (layer "Edge.Cuts") (width 0.1))
   (gr_line (start 108 33) (end 108 60.5) (layer "Edge.Cuts") (width 0.1))
-  (gr_text "Solar System\nBell Box" (at 75 57) (layer "B.SilkS")
+  (gr_text "Solar System\nBell2" (at 75 57) (layer "B.SilkS")
     (effects (font (size 1 1) (thickness 0.15)) (justify right mirror))
   )
