File: KiCad/Relay.kicad_pcb (KiCad board)
At the start: 2 copper layers, 46.5 x 30 mm, 40 parts, among them J1 USB-C, J10 O8, J2 POWER, J3 O1, J4 O2, J5 O3, J6 O4, J7 O5, J8 O6, J9 O7, U1 ESP32-PICO-MINI-02, U2 FT231XQ, U3 ISL89410, U4 ISL89410, U5 ISL89410, U6 ISL89410, U7 LMR16006+FB, U8 AA, U9 QR

Commit message: PSU
Parts:
- moved C2 15.5 mm to (110.5, 55.5), turned to 90 degrees
- moved C3 12.7 mm to (111.7, 58.8), turned to 90 degrees
- moved C4 11.2 mm to (118.0, 58.8), turned to 90 degrees
- moved D3 6.45 mm to (114.8, 58.4)
- moved L1 6.25 mm to (116.5, 55.2)
Changed lines of the file:
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@@
   )
   (footprint "RevK:Hidden" (layer "F.Cu")
-    (at 114.61 70.45)
+    (at 110.45 55.5 90)
     (property "Note" "X7R or X5R 0603")
     (property "Part No" "")
@@
     (property "Sheetname" "")
     (attr smd)
-    (fp_text reference "C2" (at 0 -0.8) (layer "F.SilkS") hide
-      (effects (font (size 0.5 0.5) (thickness 0.08)))
-    )
-    (fp_text value "0.1uF" (at 0 0.75) (layer "F.Fab")
-      (effects (font (size 0.5 0.5) (thickness 0.08)))
-    )
-    (fp_text user "${REFERENCE}" (at 0 -0.8) (layer "F.Fab")
+    (fp_text reference "C2" (at 0 -0.8 90) (layer "F.SilkS") hide
+      (effects (font (size 0.5 0.5) (thickness 0.08)))
+    )
+    (fp_text value "0.1uF" (at 0 0.75 90) (layer "F.Fab")
+      (effects (font (size 0.5 0.5) (thickness 0.08)))
+    )
+    (fp_text user "${REFERENCE}" (at 0 -0.8 90) (layer "F.Fab")
       (effects (font (size 0.5 0.5) (thickness 0.08)))
     )
@@
   )
   (footprint "RevK:Hidden" (layer "F.Cu")
-    (at 116.73 70.45)
+    (at 111.7 58.8 90)
     (property "Note" "0603 or 0805")
     (property "Part No" "")
@@
     (property "Sheetname" "")
     (attr smd)
-    (fp_text reference "C3" (at 0 -0.8) (layer "F.SilkS") hide
-      (effects (font (size 0.5 0.5) (thickness 0.08)))
-    )
-    (fp_text value "2.2uF" (at 0 0.75) (layer "F.Fab")
-      (effects (font (size 0.5 0.5) (thickness 0.08)))
-    )
-    (fp_text user "${REFERENCE}" (at 0 -0.8) (layer "F.Fab")
+    (fp_text reference "C3" (at 0 -0.8 90) (layer "F.SilkS") hide
+      (effects (font (size 0.5 0.5) (thickness 0.08)))
+    )
+    (fp_text value "2.2uF" (at 0 0.75 90) (layer "F.Fab")
+      (effects (font (size 0.5 0.5) (thickness 0.08)))
+    )
+    (fp_text user "${REFERENCE}" (at 0 -0.8 90) (layer "F.Fab")
       (effects (font (size 0.5 0.5) (thickness 0.08)))
     )
@@
   )
   (footprint "RevK:Hidden" (layer "F.Cu")
-    (at 111.75 52.75)
+    (at 114.83 58.42)
     (property "Manufacturer" "Bourns")
     (property "Note" "")
@@
   )
   (footprint "RevK:Hidden" (layer "F.Cu")
-    (at 111.75 51.13)
+    (at 116.45 55.25)
     (property "Manufacturer" "Laird")
     (property "Note" "")
@@
   )
   (footprint "RevK:Hidden" (layer "F.Cu")
-    (at 111.75 49.51)
+    (at 117.95 58.8 90)
     (property "Note" "0603 or 0805")
     (property "Part No" "")
@@
     (property "Sheetname" "")
     (attr smd)
-    (fp_text reference "C4" (at 0 -0.8) (layer "F.SilkS") hide
-      (effects (font (size 0.5 0.5) (thickness 0.08)))
-    )
-    (fp_text value "10uF" (at 0 0.75) (layer "F.Fab")
-      (effects (font (size 0.5 0.5) (thickness 0.08)))
-    )
-    (fp_text user "${REFERENCE}" (at 0 -0.8) (layer "F.Fab")
-      (effects (font (size 0.5 0.5) (thickness 0.08)))
-    )
+    (fp_text reference "C4" (at 0 -0.8 90) (layer "F.SilkS") hide
+      (effects (font (size 0.5 0.5) (thickness 0.08)))
+    )
+    (fp_text value "10uF" (at 0 0.75 90) (layer "F.Fab")
+      (effects (font (size 0.5 0.5) (thickness 0.08)))
+    )
+    (fp_text user "${REFERENCE}" (at 0 -0.8 90) (layer "F.Fab")
+      (effects (font (size 0.5 0.5) (thickness 0.08)))
+    )

Commit message: Tidy
Parts:
- moved AJK1 1.13 mm to (103.4, 35.2)
Changed lines of the file:
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@@
   )
   (footprint "RevK:AJK" (layer "B.Cu")
-    (at 104.25 36 180)
+    (at 103.4 35.25 180)
     (property "Note" "Non part, PCB printed")
     (property "Sheetfile" "Relay.kicad_sch")
