File: KiCad/Relay10.kicad_pcb (KiCad board)
At the start: 2 copper layers, 46.5 x 30 mm, 41 parts, among them J1 USB-C, J10 O8, J11 O1, J2 POWER, J3 O1, J4 O2, J5 O3, J6 O4, J7 O5, J8 O6, J9 O7, U1 ESP32-PICO-MINI-02, U2 FT231XQ, U3 ISL89410, U4 ISL89410, U5 ISL89410, U6 ISL89410, U7 LMR16006+FB, U8 AA, U9 QR

Commit message: Relay 10
Parts:
- added J12: O10, RevK:Molex_MiniSPOX_H2RA, F.Cu at (88.2, 34.2)
- added U5: ISL89410, Package_SO:SO-8_3.9x4.9mm_P1.27mm, F.Cu at (93.2, 36.8)
- J11: value O1 -> O9
- moved AJK1 23.0 mm to (115.4, 43.6)
- moved R8 23.0 mm to (116.0, 35.2), turned to 180 degrees
- moved R9 23.0 mm to (116.0, 34.0), turned to 180 degrees
- moved D1 23.0 mm to (116.0, 32.3), turned to 180 degrees
- moved R10 23.0 mm to (116.0, 36.5), turned to 180 degrees
- moved J11 11.6 mm to (121.3, 26.8), turned to 90 degrees
- moved U9 8.50 mm to (115.9, 37.0)
- moved J3 7.50 mm to (88.2, 26.8)
- moved J5 7.50 mm to (88.2, 56.8)
- moved J6 7.50 mm to (88.2, 49.2)
- moved R1 1.75 mm to (97.2, 32.5), turned to -90 degrees
- renumbered U9 to U10, U5 to U6, U6 to U7, U7 to U8, U8 to U9
Connections:
- J11 pad 2: I1 -> O9
- U1 pad 18: unconnected-(U1-Pad18) -> OUT10
- U1 pad 20: unconnected-(U1-Pad20) -> OUT9
- U1 pad 21: I1 -> unconnected-(U1-Pad21)
- U1 pad 33: G -> B
- U1 pad 35: B -> G
Routing:
- net O9: track 0.00 -> 40.2 mm, vias 0 -> 1
- net +3V3: track 58.5 -> 81.9 mm, vias 3 -> 4
- net G: track 25.5 -> 5.02 mm, vias 2 -> 0
- net I1: track 18.8 -> 0.00 mm, vias 1 -> 0
- net R: track 20.9 -> 5.25 mm, vias 2 -> 0
- net B: track 20.8 -> 5.52 mm, vias 2 -> 0
- net OUT9: track 0.00 -> 14.0 mm, vias 0 -> 2
- net OUT10: track 0.00 -> 12.3 mm, vias 0 -> 2
- net O4: track 13.9 -> 2.96 mm
- net EN: track 12.8 -> 22.5 mm, vias 2 -> 3
- net O1: track 6.44 -> 14.8 mm
- net +12V: track 62.3 -> 69.9 mm
- net O3: track 8.08 -> 15.5 mm
- net O10: track 0.00 -> 3.53 mm
- net Net-(D1-Pad3): track 4.54 -> 1.23 mm
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Other:
- board size 46.5 x 30 mm -> 46.5 x 37.5 mm
- board text added: "13"
- board text added: "14"
- board text added: "RGB: 22/21/19"
- board text removed: "15"
- board text removed: "Input"
- board text removed: "RGB: 22/19/21"

Commit message: Tidy text
Other:
- board text added: "Output Board"
- board text removed: "Relay Board"
Changed lines of the file:
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@@
   (paper "A4")
   (title_block
-    (title "Bell box controller")
+    (title "Output board (10)")
     (date "${DATE}")
-    (rev "2")
+    (rev "1")
     (company "Adrian Kennard, Andrews & Arnold Ltd")
   )
@@
       (layer "F.SilkS" (type "Top Silk Screen"))
       (layer "F.Paste" (type "Top Solder Paste"))
-      (layer "F.Mask" (type "Top Solder Mask") (thickness 0.01))
+      (layer "F.Mask" (type "Top Solder Mask") (color "Purple") (thickness 0.01))
       (layer "F.Cu" (type "copper") (thickness 0.035))
       (layer "dielectric 1" (type "core") (thickness 1.51) (material "FR4") (epsilon_r 4.5) (loss_tangent 0.02))
       (layer "B.Cu" (type "copper") (thickness 0.035))
-      (layer "B.Mask" (type "Bottom Solder Mask") (thickness 0.01))
+      (layer "B.Mask" (type "Bottom Solder Mask") (color "Purple") (thickness 0.01))
       (layer "B.Paste" (type "Bottom Solder Paste"))
       (layer "B.SilkS" (type "Bottom Silk Screen"))
@@
     (effects (font (size 0.8 0.8) (thickness 0.1)) (justify mirror))
   )
-  (gr_text "Relay\nBoard" (at 114.75 55.25) (layer "B.SilkS")
+  (gr_text "Output\nBoard" (at 114.75 55.25) (layer "B.SilkS")
     (effects (font (size 1 1) (thickness 0.15)) (justify mirror))
   )
@@
     (effects (font (size 0.75 0.75) (thickness 0.1)))
   )
-  (gr_text "Relay\nBoard" (at 109.25 45.25) (layer "F.SilkS")
+  (gr_text "Output\nBoard" (at 109.25 45.25) (layer "F.SilkS")
     (effects (font (size 1 1) (thickness 0.15)))
   )
