File: KiCad/Relay10.kicad_sch (KiCad schematic)
At the start: 41 parts, among them J1 USB-C, J10 O8, J11 O1, J2 POWER, J3 O1, J4 O2, J5 O3, J6 O4, J7 O5, J8 O6, J9 O7, U1 ESP32-PICO-MINI-02, U2 FT231XQ, U3 ISL89410, U4 ISL89410, U5 ISL89410, U6 ISL89410, U7 LMR16006+FB, U8 AA, U9 QR

Commit message: Relay 10
Parts:
- added J12: O10, RevK:Molex_MiniSPOX_H2RA, symbol Connector_Generic:Conn_01x02
- added U5: ISL89410, Package_SO:SO-8_3.9x4.9mm_P1.27mm, symbol Driver_FET:EL7202CN
- J11: value O1 -> O9
- renumbered U9 to U10, U5 to U6, U6 to U7, U7 to U8, U8 to U9
Connections:
- net +12V: now also U5.6 (V+)
- net B: now also U1.33 (IO19); no longer U1.35 (IO21)
- net G: now also U1.35 (IO21); no longer U1.33 (IO19)
- net GND: now also J12.1 (Pin_1), U5.3 (GND)
- net OUT10: now reaches U1.18 (IO14)
- net OUT10: now also U5.2 (IN_A)
- net OUT9: now reaches U1.20 (IO13)
- net OUT9: now also U5.4 (IN_B)
- net I1: no longer names the net of U1.21 (IO15)
- net I1: no longer J11.2 (Pin_2)
- new net O10: J12.2 (Pin_2), U5.7 (OUT_A)
- new net O9: J11.2 (Pin_2), U5.5 (OUT_B)

Commit message: Tidy text
Other:
- title: bell box control -> Output board (10)
Changed lines of the file:
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@@
   (paper "A4")
   (title_block
-    (title "bell box control")
+    (title "Output board (10)")
     (date "${DATE}")
-    (rev "2")
+    (rev "1")
     (company "Adrian Kennard Andrews & Arnold Ltd")
     (comment 1 "@TheRealRevK")
