File: KiCad/Relay8.kicad_pcb (KiCad board)
At the start: 2 copper layers, 46.5 x 30 mm, 41 parts, among them J1 USB-C, J10 O8, J11 O1, J2 POWER, J3 O1, J4 O2, J5 O3, J6 O4, J7 O5, J8 O6, J9 O7, U1 ESP32-PICO-MINI-02, U2 FT231XQ, U3 ISL89410, U4 ISL89410, U5 ISL89410, U6 ISL89410, U7 LMR16006+FB, U8 AA, U9 QR

Commit message: Tidy text
Other:
- board text added: "Output Board"
- board text removed: "Relay Board"
Changed lines of the file:
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@@
   (paper "A4")
   (title_block
-    (title "Bell box controller")
+    (title "Output board (8)")
     (date "${DATE}")
-    (rev "2")
+    (rev "1")
     (company "Adrian Kennard, Andrews & Arnold Ltd")
   )
@@
     (fp_line (start -2.7 -1.3) (end -3.7 -0.3) (layer "F.Fab") (width 0.12))
     (fp_line (start 3.7 -1.3) (end 3.7 6.6) (layer "F.Fab") (width 0.12))
-    (pad "1" thru_hole roundrect (at -1.25 0 270) (size 1.7 1.85) (drill 0.85) (layers *.Cu *.Mask) (roundrect_rratio 0.147059)
+    (pad "1" thru_hole roundrect (at -1.25 0 270) (size 1.7 1.85) (drill 0.85) (layers *.Cu *.Mask) (roundrect_rratio 0.1470588235)
       (net 1 "GND") (pinfunction "Pin_1") (pintype "passive"))
     (pad "2" thru_hole oval (at 1.25 0 270) (size 1.7 1.85) (drill 0.85) (layers *.Cu *.Mask)
@@
     (fp_line (start 3.7 -1.3) (end 3.7 6.6) (layer "F.Fab") (width 0.12))
     (fp_line (start 0 2) (end -1 3) (layer "F.Fab") (width 0.12))
-    (pad "1" thru_hole roundrect (at -1.25 0 270) (size 1.7 1.85) (drill 0.85) (layers *.Cu *.Mask) (roundrect_rratio 0.147059)
+    (pad "1" thru_hole roundrect (at -1.25 0 270) (size 1.7 1.85) (drill 0.85) (layers *.Cu *.Mask) (roundrect_rratio 0.1470588235)
       (net 1 "GND") (pinfunction "Pin_1") (pintype "passive"))
     (pad "2" thru_hole oval (at 1.25 0 270) (size 1.7 1.85) (drill 0.85) (layers *.Cu *.Mask)
@@
     (fp_line (start 0 5) (end 0 2) (layer "F.Fab") (width 0.12))
     (fp_line (start -3.7 -1.3) (end 3.7 -1.3) (layer "F.Fab") (width 0.12))
-    (pad "1" thru_hole roundrect (at -1.25 0 90) (size 1.7 1.85) (drill 0.85) (layers *.Cu *.Mask) (roundrect_rratio 0.147059)
+    (pad "1" thru_hole roundrect (at -1.25 0 90) (size 1.7 1.85) (drill 0.85) (layers *.Cu *.Mask) (roundrect_rratio 0.1470588235)
       (net 1 "GND") (pinfunction "Pin_1") (pintype "passive"))
     (pad "2" thru_hole oval (at 1.25 0 90) (size 1.7 1.85) (drill 0.85) (layers *.Cu *.Mask)
@@
     (fp_line (start 3.7 6.6) (end -3.7 6.6) (layer "F.Fab") (width 0.12))
     (fp_line (start 0 2) (end 1 3) (layer "F.Fab") (width 0.12))
-    (pad "1" thru_hole roundrect (at -1.25 0 180) (size 1.7 1.85) (drill 0.85) (layers *.Cu *.Mask) (roundrect_rratio 0.147059)
+    (pad "1" thru_hole roundrect (at -1.25 0 180) (size 1.7 1.85) (drill 0.85) (layers *.Cu *.Mask) (roundrect_rratio 0.1470588235)
       (net 1 "GND") (pinfunction "Pin_1") (pintype "passive"))
     (pad "2" thru_hole oval (at 1.25 0 180) (size 1.7 1.85) (drill 0.85) (layers *.Cu *.Mask)
@@
     (fp_line (start -3.7 6.6) (end -3.7 -1.3) (layer "F.Fab") (width 0.12))
     (fp_line (start 3.7 6.6) (end -3.7 6.6) (layer "F.Fab") (width 0.12))
-    (pad "1" thru_hole roundrect (at -1.25 0) (size 1.7 1.85) (drill 0.85) (layers *.Cu *.Mask) (roundrect_rratio 0.147059)
+    (pad "1" thru_hole roundrect (at -1.25 0) (size 1.7 1.85) (drill 0.85) (layers *.Cu *.Mask) (roundrect_rratio 0.1470588235)
       (net 1 "GND") (pinfunction "GND") (pintype "power_in"))
     (pad "2" thru_hole oval (at 1.25 0) (size 1.7 1.85) (drill 0.85) (layers *.Cu *.Mask)
@@
     (fp_line (start 3.7 -1.3) (end 3.7 6.6) (layer "F.Fab") (width 0.12))
     (fp_line (start 0 5) (end 0 2) (layer "F.Fab") (width 0.12))
-    (pad "1" thru_hole roundrect (at -1.25 0 270) (size 1.7 1.85) (drill 0.85) (layers *.Cu *.Mask) (roundrect_rratio 0.147059)
+    (pad "1" thru_hole roundrect (at -1.25 0 270) (size 1.7 1.85) (drill 0.85) (layers *.Cu *.Mask) (roundrect_rratio 0.1470588235)
       (net 1 "GND") (pinfunction "Pin_1") (pintype "passive"))
     (pad "2" thru_hole oval (at 1.25 0 270) (size 1.7 1.85) (drill 0.85) (layers *.Cu *.Mask)
@@
     (fp_line (start 3.7 6.6) (end -3.7 6.6) (layer "F.Fab") (width 0.12))
     (fp_line (start 0 2) (end -1 3) (layer "F.Fab") (width 0.12))
-    (pad "1" thru_hole roundrect (at -1.25 0 90) (size 1.7 1.85) (drill 0.85) (layers *.Cu *.Mask) (roundrect_rratio 0.147059)
+    (pad "1" thru_hole roundrect (at -1.25 0 90) (size 1.7 1.85) (drill 0.85) (layers *.Cu *.Mask) (roundrect_rratio 0.1470588235)
       (net 1 "GND") (pinfunction "Pin_1") (pintype "passive"))
     (pad "2" thru_hole oval (at 1.25 0 90) (size 1.7 1.85) (drill 0.85) (layers *.Cu *.Mask)
@@
     (fp_line (start -3.7 -1.3) (end 3.7 -1.3) (layer "F.Fab") (width 0.12))
     (fp_line (start 3.7 6.6) (end -3.7 6.6) (layer "F.Fab") (width 0.12))
-    (pad "1" thru_hole roundrect (at -1.25 0 90) (size 1.7 1.85) (drill 0.85) (layers *.Cu *.Mask) (roundrect_rratio 0.147059)
+    (pad "1" thru_hole roundrect (at -1.25 0 90) (size 1.7 1.85) (drill 0.85) (layers *.Cu *.Mask) (roundrect_rratio 0.1470588235)
       (net 1 "GND") (pinfunction "Pin_1") (pintype "passive"))
     (pad "2" thru_hole oval (at 1.25 0 90) (size 1.7 1.85) (drill 0.85) (layers *.Cu *.Mask)
@@
     (fp_line (start 0 2) (end 1 3) (layer "F.Fab") (width 0.12))
     (fp_line (start 0 5) (end 0 2) (layer "F.Fab") (width 0.12))
-    (pad "1" thru_hole roundrect (at -1.25 0 90) (size 1.7 1.85) (drill 0.85) (layers *.Cu *.Mask) (roundrect_rratio 0.147059)
+    (pad "1" thru_hole roundrect (at -1.25 0 90) (size 1.7 1.85) (drill 0.85) (layers *.Cu *.Mask) (roundrect_rratio 0.1470588235)
       (net 1 "GND") (pinfunction "Pin_1") (pintype "passive"))
     (pad "2" thru_hole oval (at 1.25 0 90) (size 1.7 1.85) (drill 0.85) (layers *.Cu *.Mask)
@@
     (fp_line (start -3.7 -1.3) (end 3.7 -1.3) (layer "F.Fab") (width 0.12))
     (fp_line (start -3.7 6.6) (end -3.7 -1.3) (layer "F.Fab") (width 0.12))
-    (pad "1" thru_hole roundrect (at -1.25 0 270) (size 1.7 1.85) (drill 0.85) (layers *.Cu *.Mask) (roundrect_rratio 0.147059)
+    (pad "1" thru_hole roundrect (at -1.25 0 270) (size 1.7 1.85) (drill 0.85) (layers *.Cu *.Mask) (roundrect_rratio 0.1470588235)
       (net 1 "GND") (pinfunction "Pin_1") (pintype "passive"))
     (pad "2" thru_hole oval (at 1.25 0 270) (size 1.7 1.85) (drill 0.85) (layers *.Cu *.Mask)
@@
     (effects (font (size 0.8 0.8) (thickness 0.1)) (justify mirror))
   )
-  (gr_text "Relay\nBoard" (at 114.75 55.25) (layer "B.SilkS")
+  (gr_text "Output\nBoard" (at 114.75 55.25) (layer "B.SilkS")
     (effects (font (size 1 1) (thickness 0.15)) (justify mirror))
   )
@@
     (effects (font (size 0.75 0.75) (thickness 0.1)))
   )
-  (gr_text "Relay\nBoard" (at 109.25 43.75) (layer "F.SilkS")
+  (gr_text "Output\nBoard" (at 109.25 43.75) (layer "F.SilkS")
     (effects (font (size 1 1) (thickness 0.15)))
   )
