File: KiCad/Relay8.kicad_sch (KiCad schematic)
At the start: 41 parts, among them J1 USB-C, J10 O8, J11 O1, J2 POWER, J3 O1, J4 O2, J5 O3, J6 O4, J7 O5, J8 O6, J9 O7, U1 ESP32-PICO-MINI-02, U2 FT231XQ, U3 ISL89410, U4 ISL89410, U5 ISL89410, U6 ISL89410, U7 LMR16006+FB, U8 AA, U9 QR

Commit message: Relay 10
Parts:
- J11: value O1 -> I1
Changed lines of the file:
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@@
       (effects (font (size 1.27 1.27)) (justify left))
     )
-    (property "Value" "O1" (id 1) (at 245.872 137.5922 0)
+    (property "Value" "I1" (id 1) (at 245.872 137.5922 0)
       (effects (font (size 1.27 1.27)) (justify left))
     )
@@
     )
     (path "/515530bd-0566-4c2d-8cd0-a23d5fcc09ed"
-      (reference "J11") (unit 1) (value "O1") (footprint "RevK:Molex_MiniSPOX_H2RA")
+      (reference "J11") (unit 1) (value "I1") (footprint "RevK:Molex_MiniSPOX_H2RA")
     )
     (path "/00000000-0000-0000-0000-0000610fe01a"

Commit message: Tidy text
Other:
- title: bell box control -> Output board (8)
Changed lines of the file:
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@@
   (paper "A4")
   (title_block
-    (title "bell box control")
+    (title "Output board (8)")
     (date "${DATE}")
-    (rev "2")
+    (rev "1")
     (company "Adrian Kennard Andrews & Arnold Ltd")
     (comment 1 "@TheRealRevK")
