File: PCB/Keypad2/Keypad2.kicad_pcb (KiCad board)
At the start: 2 copper layers, 13.2 x 29 mm, 21 parts, among them J1 Keypad, J2 Shelly, U1 SP3485, U2 ESP32-PICO-MINI-02, U3 LMR16006+FB, U4 QR

Commit message: PCb tweak
Parts:
- removed C2: 0.1uF, RevK:C_0603_
- removed C3: 2.2uF, RevK:C_0805_
- removed C4: 10uF, RevK:C_0805_
- removed D2: Schottky, RevK:D_1206_
- removed L1: 6.8uH, RevK:L_4x4_
- removed U3: LMR16006+FB, RevK:SOT-23-Thin-6-Reg
- added C6: 100nF, RevK:C_0603_, F.Cu at (171.1, 108.4)
- added C7: 2.2uF, RevK:C_0805_, F.Cu at (167.8, 109.6)
- added C8: 10uF, RevK:C_0805_, F.Cu at (167.8, 115.9)
- added D3: Schottky, RevK:D_1206_, F.Cu at (168.2, 112.7)
- added L2: 6.8uH, RevK:L_4x4_, F.Cu at (171.4, 114.4)
- added U5: LMR16006YDDCR, RevK:SOT-23-Thin-6-Reg, F.Cu at (171.4, 110.5)
Routing:
- net GND: track 48.7 -> 40.0 mm
Other:
- board text added: "${DATE}"
- board text added: "A"
- board text added: "B"
- board text added: "DC"
- board text added: "DE:13 Tx:14 Rx:15 RGB:25/26/27"
- board text added: "⏚"

Commit message: Tidy for production
Parts:
- removed C6: 100nF, RevK:C_0603_
- removed C7: 2.2uF, RevK:C_0805_
- removed C8: 10uF, RevK:C_0805_
- removed D3: Schottky, RevK:D_1206_
- removed L2: 6.8uH, RevK:L_4x4_
- removed R5: 100k 1% or 0R, RevK:R_0603
- removed R6: 30k 1% or NF, RevK:R_0603
- removed U5: LMR16006YDDCR, RevK:SOT-23-Thin-6-Reg
- added C2: 100nF, RevK:C_0603_, F.Cu at (171.2, 108.4)
- added C3: 2.2uF, RevK:C_0805_, F.Cu at (167.8, 109.7)
- added C4: 10uF, RevK:C_0805_, F.Cu at (167.8, 115.9)
- added D2: LED_BARG, RevK:MHS190RGBCT, F.Cu at (162.2, 107.9)
- added L1: 6.8uH, RevK:L_4x4_, F.Cu at (171.4, 114.4)
- added R7: 100k 1%, RevK:R_0603, F.Cu at (171.5, 106.6)
- added R8: 30k 1%, RevK:R_0603, F.Cu at (173.4, 107.4)
- added U3: LMR16006YDDCR, RevK:SOT-23-Thin-6-Reg, F.Cu at (171.4, 110.5)
- D1: value LED_RGBA -> Schottky; footprint RevK:LED-RGB-1.6x1.6 -> RevK:D_1206_
- moved D1 8.25 mm to (168.2, 112.8), turned to -90 degrees
Connections:
- R2 pad 1: Net-(D1-RK) -> Net-(D2-RK)
- R3 pad 1: Net-(D1-GK) -> Net-(D2-GK)
- R4 pad 1: Net-(D1-BK) -> Net-(D2-BK)
Routing:
- net Net-(D1-BK): track 5.63 -> 0.00 mm
- net Net-(D2-BK): track 0.00 -> 4.82 mm
- net Net-(D1-GK): track 4.30 -> 0.00 mm
- net +3V3: track 57.1 -> 60.9 mm
- net Net-(U5-FB): track 3.58 -> 0.00 mm
- net Net-(U3-FB): track 0.00 -> 3.58 mm
- net Net-(D2-GK): track 0.00 -> 3.46 mm
- net Net-(D2-RK): track 0.00 -> 1.85 mm
- net Net-(D1-RK): track 1.17 -> 0.00 mm

Commit message: Cap change
Parts:
- C1: value 10nF -> 1uF
Changed lines of the file:
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@@
+        (effects (font (size 0.5 0.5) (thickness 0.08)))
+    )
+    (fp_text user "D" (at -0.8 0 -90 unlocked) (layer "F.Fab")
         (effects (font (size 0.5 0.5) (thickness 0.08)))
     )
     (fp_text user "${REFERENCE}" (at 0 -1.2 90) (layer "F.Fab")
-        (effects (font (size 0.5 0.5) (thickness 0.08)))
-    )
-    (fp_text user "D" (at -0.8 0 -90 unlocked) (layer "F.Fab")
         (effects (font (size 0.5 0.5) (thickness 0.08)))
     )
@@
         (effects (font (size 0.5 0.5) (thickness 0.1)))
     )
+    (fp_text user "From PCB" (at 11 -8.2 90 unlocked) (layer "F.Fab")
+        (effects (font (size 0.5 0.5) (thickness 0.1)))
+    )
+    (fp_text user "Max 2mm" (at -8.1 -8.4 90 unlocked) (layer "F.Fab")
+        (effects (font (size 0.5 0.5) (thickness 0.1)))
+    )
+    (fp_text user "From edge" (at -7.3 -8.4 90 unlocked) (layer "F.Fab")
+        (effects (font (size 0.5 0.5) (thickness 0.1)))
+    )
+    (fp_text user "Max 1mm" (at 0 -11.5 unlocked) (layer "F.Fab")
+        (effects (font (size 0.5 0.5) (thickness 0.1)))
+    )
     (fp_text user "ANTENNA" (at -3 -7.7) (layer "F.Fab")
         (effects (font (size 0.787402 0.787402) (thickness 0.15)))
     )
-    (fp_text user "Max 2mm" (at -8.1 -8.4 90 unlocked) (layer "F.Fab")
-        (effects (font (size 0.5 0.5) (thickness 0.1)))
-    )
-    (fp_text user "From edge" (at -7.3 -8.4 90 unlocked) (layer "F.Fab")
-        (effects (font (size 0.5 0.5) (thickness 0.1)))
-    )
-    (fp_text user "From PCB" (at 11 -8.2 90 unlocked) (layer "F.Fab")
-        (effects (font (size 0.5 0.5) (thickness 0.1)))
-    )
-    (fp_text user "Max 1mm" (at 0 -11.5 unlocked) (layer "F.Fab")
-        (effects (font (size 0.5 0.5) (thickness 0.1)))
-    )
-    (fp_line (start -6.5 -5.1) (end -6.5 -4.6)
-      (stroke (width 0.2) (type solid)) (layer "F.SilkS"))
-    (fp_line (start -6.5 4.6) (end -6.5 5.5)
-      (stroke (width 0.2) (type solid)) (layer "F.SilkS"))
-    (fp_line (start -6.5 5.5) (end -5.6 5.5)
-      (stroke (width 0.2) (type solid)) (layer "F.SilkS"))
-    (fp_line (start 6.5 -5.1) (end 6.5 -4.6)
-      (stroke (width 0.2) (type solid)) (layer "F.SilkS"))
-    (fp_line (start 6.5 4.6) (end 6.5 5.5)
-      (stroke (width 0.2) (type solid)) (layer "F.SilkS"))
-    (fp_line (start 6.5 5.5) (end 5.6 5.5)
-      (stroke (width 0.2) (type solid)) (layer "F.SilkS"))
     (fp_line (start -6.6 -11) (end -6.6 5.6)
       (stroke (width 0.05) (type solid)) (layer "F.CrtYd"))
@@
         (effects (font (size 0.5 0.5) (thickness 0.1)) (justify left))
     )
-    (fp_text user "LMR" (at -1.4 -0.3 -90 unlocked) (layer "F.Fab")
+    (fp_text user "16006" (at -1.4 0.45 -90 unlocked) (layer "F.Fab")
         (effects (font (size 0.5 0.5) (thickness 0.1)) (justify left))
     )
@@
         (effects (font (size 0.5 0.5) (thickness 0.1)) (justify right))
     )
-    (fp_text user "16006" (at -1.4 0.45 -90 unlocked) (layer "F.Fab")
+    (fp_text user "LMR" (at -1.4 -0.3 -90 unlocked) (layer "F.Fab")
         (effects (font (size 0.5 0.5) (thickness 0.1)) (justify left))
     )
@@
         (effects (font (size 0.5 0.5) (thickness 0.08)))
     )
+    (fp_text user "${REFERENCE}" (at 0 -1.075) (layer "F.Fab")
+        (effects (font (size 0.5 0.5) (thickness 0.08)))
+    )
     (fp_text user "C" (at -0.5 0 unlocked) (layer "F.Fab")
-        (effects (font (size 0.5 0.5) (thickness 0.08)))
-    )
-    (fp_text user "${REFERENCE}" (at 0 -1.075) (layer "F.Fab")
         (effects (font (size 0.5 0.5) (thickness 0.08)))
     )
@@
         (effects (font (size 0.5 0.5) (thickness 0.08)))
     )
+    (fp_text user "${REFERENCE}" (at 0 -1) (layer "F.Fab")
+        (effects (font (size 0.5 0.5) (thickness 0.08)))
+    )
     (fp_text user "C" (at -0.5 0 unlocked) (layer "F.Fab")
-        (effects (font (size 0.5 0.5) (thickness 0.08)))
-    )
-    (fp_text user "${REFERENCE}" (at 0 -1) (layer "F.Fab")
         (effects (font (size 0.5 0.5) (thickness 0.08)))
     )
@@
         (effects (font (size 0.5 0.5) (thickness 0.08)))
     )
-    (fp_text value "10nF" (at 0 0) (layer "F.Fab")
+    (fp_text value "1uF" (at 0 0) (layer "F.Fab")
         (effects (font (size 0.4 0.4) (thickness 0.08)))
     )
@@
         (effects (font (size 1 1) (thickness 0.15)) (justify mirror))
     )
+    (fp_text user "↑3" (at -3.37 0.8 315 unlocked) (layer "B.SilkS")
+        (effects (font (size 0.5 0.5) (thickness 0.08)) (justify mirror))
+    )
     (fp_text user "0" (at 1.71 0.8 315 unlocked) (layer "B.SilkS")
         (effects (font (size 0.5 0.5) (thickness 0.08)) (justify mirror))
     )
-    (fp_text user "↑3" (at -3.37 0.8 315 unlocked) (layer "B.SilkS")
+    (fp_text user "⏚" (at 4.25 0.8 315 unlocked) (layer "B.SilkS")
         (effects (font (size 0.5 0.5) (thickness 0.08)) (justify mirror))
     )
@@
         (effects (font (size 0.5 0.5) (thickness 0.08)) (justify mirror))
     )
-    (fp_text user "⏚" (at 4.25 0.8 315 unlocked) (layer "B.SilkS")
-        (effects (font (size 0.5 0.5) (thickness 0.08)) (justify mirror))
-    )

Commit message: Silkscreen
Other:
- board text added: "DE/RE:13 Tx:14 Rx:15 RGB:25/26/27"
- board text removed: "DE:13 Tx:14 Rx:15 RGB:25/26/27"
