File: PCB/Access1/Access.kicad_sch (KiCad schematic)
At the start: 69 parts, among them J1 USB-C, J2 RFID, J3 INPUTS, J5 POWER, J6 DOOR2, J7 DOOR1, J8 Shelly, Q2 PMF250XNEX, SW1 ESE13V01D, U1 MD8942, U10 ESP32-S3-MINI-1, U2 MD8942, U3 G3VM-41GR8, U7 QR, U8 G3VM-41GR8, U9 AA

Commit message: Reworked
Parts:
- removed C1, C21: 10uF 50V, RevK:C_0603_, symbol RevK:Hidden
- removed C15, C22: 10uF 6.3V, RevK:C_0603_, symbol RevK:Hidden
- removed C16, C23: 100nF, RevK:C_0603_, symbol RevK:Hidden
- removed C18: 100nF, RevK:C_0402, symbol Device:C
- removed C19: 22uF, RevK:C_0402, symbol Device:C
- removed C20: 1uF, RevK:C_0402, symbol Device:C
- removed D6: RGB, RevK:LED-RGB-1.6x1.6, symbol Device:LED_RGBA
- removed J8: Shelly, RevK:Shelly, symbol RevK:Shelly
- removed L3, L4: 10uH, RevK:L_4x4_, symbol RevK:Hidden
- removed PCB1: 70x70, RevK:PCB7070, symbol RevK:PCB
- removed R1, R14: 124k, RevK:R_0402_, symbol RevK:Hidden
- removed R15: 39k2, RevK:R_0402_, symbol RevK:Hidden
- removed R2: 23k2, RevK:R_0402_, symbol RevK:Hidden
- removed R26: 10K, RevK:R_0402, symbol Device:R
- removed R27: 1M, RevK:R_0402_, symbol RevK:Hidden
- removed U1, U2: MD8942, RevK:SOT-23-6-MD8942, symbol RevK:MD89420-RegBlock
- removed U10: ESP32-S3-MINI-1, RevK:ESP32-S3-MINI-1, symbol RevK:ESP32-S3-MINI-1-N4R2
- removed V1, V2: ~, RevK:VCUT70, symbol RevK:VCUT
- added AJK1: AJK, RevK:AJK, symbol RevK:AJK
- added C1: 0.1uF, RevK:C_0603, symbol Device:C
- added C10, C13: 2.2uF, RevK:C_0805_, symbol RevK:Hidden
- added C11, C14: 10uF, RevK:C_0805_, symbol RevK:Hidden
- added C12, C9: 100nF, RevK:C_0603_, symbol RevK:Hidden
- added C15: 1uF, RevK:C_0603, symbol Device:C
- added C16: 10nF, RevK:C_0603, symbol Device:C
- added D5: LED_BARG, RevK:MHS190RGBCT, symbol Device:LED_BARG
- added D6, D7: Schottky, RevK:D_1206_, symbol RevK:Hidden
- added J4: Shelly, RevK:Shelly, symbol RevK:Shelly
- added L1, L2: 6.8uH, RevK:L_4x4_, symbol RevK:Hidden
- added Q1: NX7002AK, Package_TO_SOT_SMD:SOT-23, symbol Device:Q_NMOS_GSD
- added R1: 10k, RevK:R_0603, symbol Device:R
- added R14, R15: 27R, RevK:R_0603, symbol Device:R
- added R17: 300R, RevK:R_0603, symbol Device:R
- added R18: 1K, RevK:R_0603, symbol Device:R
- added R19: 100R, RevK:R_0603, symbol Device:R
- added R2: 4k7, RevK:R_0603, symbol Device:R
- added R22: 100k 1%, RevK:R_0603, symbol Device:R
- added R23: 18k 1%, RevK:R_0603, symbol Device:R
- added R24: 30k 1%, RevK:R_0603, symbol Device:R
- added U1: ESP32-PICO-MINI-02, RevK:ESP32-PICO-MINI-02, symbol RevK:ESP32-PICO-MINI-02
- added U2: FT231XQ, RevK:QFN-20-1EP_4x4mm_P0.5mm_EP2.5x2.5mm, symbol RevK:FT231XQ
- added U4, U5: LMR16006XDDCR, RevK:SOT-23-Thin-6-Reg, symbol RevK:LMR16006XDDCR
- added U6: AA, RevK:AA, symbol RevK:AA
- C17: footprint RevK:C_0402 -> RevK:C_0805
- C2, C3, C4, C5, C6, C7, C8: footprint RevK:C_0402 -> RevK:C_0603
- R10, R11, R12, R13, R16, R25, R4, R5, R6, R7, R8, R9: footprint RevK:R_0402 -> RevK:R_0603
- R20: value 2K -> 100K; footprint RevK:R_0402 -> RevK:R_0603
- R21: value 220R -> 100k 1%; footprint RevK:R_0402 -> RevK:R_0603; LCSC Part # (none) -> C14675
- R3: value 680R -> 10k; footprint RevK:R_0402 -> RevK:R_0603
Connections:
- net +12V: now also R20.2, U4.5 (VIN), U5.4 (SHDN), U5.5 (VIN)
- net +3.3V: now also C1.1, C16.1, D5.2 (A), J4.3 (3V3), R1.1, R22.1, U1.3 (3V3), U2.10 (3V3OUT), U2.11 (~{RESET}), U2.12 (VCC), U2.20 (VCCIO), U5.7 (VOUT)
- net +5V: now also R21.1, U4.7 (VOUT)
- net B: now also R19.2, U1.13 (IO33); no longer R21.2
- net D+: now also R15.1, U2.8 (USBDP); no longer J1.A6 (D+), J1.B6 (D+)
- net D-: now also R14.1, U2.9 (USBDM); no longer J1.A7 (D-), J1.B7 (D-)
- net G: now also R18.2, U1.15 (IO25); no longer R20.2
- net GND: now also R3.2, C1.2, C15.1, C16.2, J4.1 (GND), Q1.2 (S), R23.1, R24.1, U1.1 (GND), U1.11 (GND), U1.14 (GND), U1.2 (GND), U1.36 (GND), U1.37 (GND), U1.38 (GND), U1.39 (GND), U1.40 (GND), U1.41 (GND), U1.42 (GND), U1.43 (GND), U1.44 (GND), U1.45 (GND), U1.46 (GND), U1.47 (GND), U1.48 (GND), U1.49 (GND), U1.50 (GND), U1.51 (GND), U1.52 (GND), U1.53 (GND), U2.13 (GND), U2.2 (~{RI}), U2.21 (GND), U2.3 (GND), U2.4 (~{DSR}), U2.5 (~{DCD}), U2.6 (~{CTS}), U4.2 (GND), U5.2 (GND)
- net IO1: now also U1.26 (IO20)
- net IO2: now also U1.27 (IO7)
- net IO3: now also U1.28 (IO8)
- net IO4: now also U1.33 (IO19)
- net IO5: now also U1.34 (IO22)
- net IO6: now also U1.35 (IO21)
- net R: now also R17.2, U1.12 (IO32); no longer R3.2
- net RELAY1: now also U1.18 (IO14)
- net RELAY2: now also U1.17 (IO27)
- net RFRX: now also U1.21 (IO15)
- net RFTX: now also U1.24 (IO4)
- net SHDN: now also Q1.1 (G), U1.20 (IO13)
- net TAMPER: now also U1.16 (IO26)
- net VBUS: now also R2.1
- net at J6.2 (Pin_2), JP1.2 (B): now also U3.4; no longer U3.3
- net at J6.3 (Pin_3): now also U3.3; no longer U3.4
- net at R3.1: now also R2.2, U2.7 (CBUS2)
- net at R20.1: now also Q1.3 (D), U4.4 (SHDN)
- net at J7.2 (Pin_2), JP2.2 (B): now also U8.4; no longer U8.3
- net at J7.3 (Pin_3): now also U8.3; no longer U8.4
- new net: J1.A6 (D+), J1.B6 (D+), R15.2
- new net: J1.A7 (D-), J1.B7 (D-), R14.2
- new net: R22.2, R24.2, U5.3 (FB)
- new net: R21.2, R23.2, U4.3 (FB)
- new net: D5.3 (RK), R17.1
- new net: D5.1 (BK), R19.1
- new net: D5.4 (GK), R18.1
- new net BOOT: J4.2 (0), U1.23 (IO0), U2.18 (~{DTR})
- new net EN: C15.2, R1.2, U1.8 (EN), U2.19 (~{RTS})
- new net I: J4.4 (Rx), U1.30 (RXD0), U2.17 (TXD)
- new net O: J4.5 (Tx), U1.31 (TXD0), U2.1 (RXD)
- no-connect marks 1 -> 13
Other:
- moved on the sheet: J3, J6, J7, JP1, JP2, R16, R25, U3, U8
