File: PCB/Access2/Access.kicad_sch (KiCad schematic)
At the start: 76 parts, among them J1 USB-C, J2 RFID, J3 INPUTS, J4 Shelly, J5 POWER, J6 DOOR2, J7 DOOR1, Q1 NX7002AK, Q2 PMF250XNEX, SW1 ESE13V01D, U1 ESP32-PICO-MINI-02, U2 FT231XQ, U3 G3VM-41GR8, U4 LMR16006XDDCR, U5 LMR16006XDDCR, U6 AA, U7 QR, U8 G3VM-41GR8, U9 AA

Commit message: Reworked
Parts:
- removed AJK1: AJK, RevK:AJK, symbol RevK:AJK
- removed C1: 0.1uF, RevK:C_0603, symbol Device:C
- removed C10, C13: 2.2uF, RevK:C_0805_, symbol RevK:Hidden
- removed C11, C14: 10uF, RevK:C_0805_, symbol RevK:Hidden
- removed C12, C9: 100nF, RevK:C_0603_, symbol RevK:Hidden
- removed C15: 1uF, RevK:C_0603, symbol Device:C
- removed C16: 10nF, RevK:C_0603, symbol Device:C
- removed D5: LED_BARG, RevK:MHS190RGBCT, symbol Device:LED_BARG
- removed D6, D7: Schottky, RevK:D_1206_, symbol RevK:Hidden
- removed D8, D9: D, RevK:D_1206, symbol Device:D
- removed J4: Shelly, RevK:Shelly, symbol RevK:Shelly
- removed L1, L2: 6.8uH, RevK:L_4x4_, symbol RevK:Hidden
- removed Q1: NX7002AK, Package_TO_SOT_SMD:SOT-23, symbol Device:Q_NMOS_GSD
- removed R1: 10k, RevK:R_0603, symbol Device:R
- removed R14, R15: 27R, RevK:R_0603, symbol Device:R
- removed R17: 300R, RevK:R_0603, symbol Device:R
- removed R18: 1K, RevK:R_0603, symbol Device:R
- removed R19: 100R, RevK:R_0603, symbol Device:R
- removed R2: 4k7, RevK:R_0603, symbol Device:R
- removed R22: 100k 1%, RevK:R_0603, symbol Device:R
- removed R23: 18k 1%, RevK:R_0603, symbol Device:R
- removed R24: 30k 1%, RevK:R_0603, symbol Device:R
- removed U1: ESP32-PICO-MINI-02, RevK:ESP32-PICO-MINI-02, symbol RevK:ESP32-PICO-MINI-02
- removed U2: FT231XQ, RevK:QFN-20-1EP_4x4mm_P0.5mm_EP2.5x2.5mm, symbol RevK:FT231XQ
- removed U4, U5: LMR16006XDDCR, RevK:SOT-23-Thin-6-Reg, symbol RevK:LMR16006XDDCR
- removed U6: AA, RevK:AA, symbol RevK:AA
- added C1, C21: 10uF 50V, RevK:C_0603_, symbol RevK:Hidden
- added C15, C22: 10uF 6.3V, RevK:C_0603_, symbol RevK:Hidden
- added C16, C23: 100nF, RevK:C_0603_, symbol RevK:Hidden
- added C18: 100nF, RevK:C_0402, symbol Device:C
- added C19: 22uF, RevK:C_0402, symbol Device:C
- added C20: 1uF, RevK:C_0402, symbol Device:C
- added D2 (x2): D, RevK:D_SOD-123, symbol Device:D
- added D6: RGB, RevK:LED-RGB-1.6x1.6, symbol Device:LED_RGBA
- added J8: Shelly, RevK:Shelly, symbol RevK:Shelly
- added L3, L4: 10uH, RevK:L_4x4_, symbol RevK:Hidden
- added PCB1: 70x70, RevK:PCB7070, symbol RevK:PCB
- added R1, R14: 124k, RevK:R_0402_, symbol RevK:Hidden
- added R15: 39k2, RevK:R_0402_, symbol RevK:Hidden
- added R2: 23k2, RevK:R_0402_, symbol RevK:Hidden
- added R26: 10K, RevK:R_0402, symbol Device:R
- added R27: 1M, RevK:R_0402_, symbol RevK:Hidden
- added U1, U2: MD8942, RevK:SOT-23-6-MD8942, symbol RevK:MD89420-RegBlock
- added U10: ESP32-S3-MINI-1, RevK:ESP32-S3-MINI-1, symbol RevK:ESP32-S3-MINI-1-N4R2
- added V1, V2: ~, RevK:VCUT70, symbol RevK:VCUT
- C17: footprint RevK:C_0805 -> RevK:C_0402
- C2, C3, C4, C5, C6, C7, C8: footprint RevK:C_0603 -> RevK:C_0402
- R10, R11, R12, R13, R16, R25, R4, R5, R6, R7, R8, R9: footprint RevK:R_0603 -> RevK:R_0402
- R20: value 100K -> 2K; footprint RevK:R_0603 -> RevK:R_0402
- R21: value 100k 1% -> 220R; footprint RevK:R_0603 -> RevK:R_0402; LCSC Part # C14675 -> (none)
- R3: value 10k -> 680R; footprint RevK:R_0603 -> RevK:R_0402
Connections:
- net +12V: now also D2.1 (K), D2.1 (K), U1.5 (VIN), U2.5 (VIN); no longer R20.2
- net +3.3V: now also C18.1, C19.1, D6.4 (A), J8.3 (3V3), R26.1, U10.3 (3V3), U2.8 (VOUT)
- net +5V: now also U1.8 (VOUT); no longer R21.1
- net B: now also R21.2, U10.7 (GPIO3)
- net D+: now also J1.A6 (D+), J1.B6 (D+), U10.24 (GPIO20)
- net D-: now also J1.A7 (D-), J1.B7 (D-), U10.23 (GPIO19)
- net DC: now also D2.2 (A)
- net G: now also R20.2, U10.5 (GPIO1)
- net GND: now also C18.2, C19.2, C20.2, J8.1 (GND), U1.2 (GND), U1.7 (GND), U10.1 (GND), U10.2 (GND), U10.42 (GND), U10.43 (GND), U10.46 (GND), U10.47 (GND), U10.48 (GND), U10.49 (GND), U10.50 (GND), U10.51 (GND), U10.52 (GND), U10.53 (GND), U10.54 (GND), U10.55 (GND), U10.56 (GND), U10.57 (GND), U10.58 (GND), U10.59 (GND), U10.60 (GND), U10.61 (GND), U10.62 (GND), U10.63 (GND), U10.64 (GND), U10.65 (GND), U2.2 (GND), U2.7 (GND); no longer R3.2
- net IO1: now also U10.32 (GPIO36)
- net IO2: now also U10.33 (GPIO37)
- net IO3: now also U10.34 (GPIO38)
- net IO4: now also U10.35 (GPIO39)
- net IO5: now also U10.36 (GPIO40)
- net IO6: now also U10.37 (GPIO41)
- net R: now also R3.2, U10.6 (GPIO2)
- net RELAY1: now also U10.12 (GPIO8)
- net RELAY2: now also U10.11 (GPIO7)
- net RFRX: now also U10.30 (GPIO48)
- net RFTX: now also U10.31 (GPIO35)
- net SHDN: now also U1.4 (EN), U10.41 (GPIO45)
- net TAMPER: now also U10.8 (GPIO4)
- net VBUS: now also D2.2 (A)
- net at U3.3: now also J6.2 (Pin_2), JP1.2 (B); no longer J6.3 (Pin_3)
- net at R20.1: now also D6.2 (GK)
- net at J7.2 (Pin_2), JP2.2 (B): now also U8.3; no longer U8.4
- net at R3.1: now also D6.1 (RK)
- net at J7.3 (Pin_3): now also U8.4; no longer U8.3
- new net: J6.3 (Pin_3), U3.4
- new net: D6.3 (BK), R21.1
- new net: J8.5 (Tx), U10.39 (GPIO43)
- new net: J8.2 (0), U10.4 (GPIO0)
- new net: J8.4 (Rx), U10.40 (GPIO44)
- new net: C20.1, R26.2, U10.45 (EN)
- no-connect marks 13 -> 1
Other:
- moved on the sheet: J3, J6, J7, JP1, JP2, R16, R25, U3, U8
