File: PCB/Access/Access.kicad_sch (KiCad schematic)
At the start: 63 parts, among them J1 USB-C, J2 RFID, J3 INPUTS, J4 USB-PROG, J5 POWER, J6 DOOR2, J7 DOOR1, J8 Shelly, Q2 PMF250XNEX, SW1 ESE13V01D, U1 MD8942, U10 ESP32-S3-MINI-1, U2 MD8942, U3 G3VM-41GR8, U8 G3VM-41GR8, U9 AA

Commit message: Tweak
Parts:
- added unit 1 of D1
- J1: footprint RevK:USC16-TR -> RevK:USB-C-Socket-H; symbol RevK:USB-C -> RevK:USB-C-Socket-H
Connections:
- net GND: now also SW1.2; no longer SW1.1
- net TAMPER: now also SW1.1; no longer SW1.2
- no-connect marks 20 -> 24
Changed lines of the file:
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@@
   (no_connect (at 38.735 72.39))
   (no_connect (at 69.215 102.87))
+  (no_connect (at 143.51 97.79))
   (no_connect (at 38.735 102.87))
   (no_connect (at 38.735 57.15))
+  (no_connect (at 151.13 102.87))
   (no_connect (at 38.735 90.17))
   (no_connect (at 38.735 62.23))
@@
   (no_connect (at 223.52 102.235))
   (no_connect (at 69.215 67.31))
+  (no_connect (at 69.215 90.17))
   (no_connect (at 38.735 95.25))
   (no_connect (at 38.735 87.63))
   (no_connect (at 38.735 54.61))
   (no_connect (at 38.735 59.69))
+  (no_connect (at 158.75 97.79))
   (no_connect (at 205.74 37.465))
   (no_connect (at 38.735 80.01))
@@
     )
   )
-  (symbol (lib_id "RevK:USB-C") (at 104.775 36.83 0) (unit 1)
+  (symbol (lib_id "RevK:USB-C-Socket-H") (at 104.775 36.83 0) (unit 1)
     (in_bom yes) (on_board yes) (dnp no)
     (property "Reference" "J1" (at 107.4928 14.8082 0)
@@
       (effects (font (size 1.27 1.27)))
     )
-    (property "Footprint" "RevK:USC16-TR" (at 108.585 36.83 0)
+    (property "Footprint" "RevK:USB-C-Socket-H" (at 104.775 16.51 0)
       (effects (font (size 1.27 1.27)) hide)
     )
-    (property "Datasheet" "https://www.usb.org/sites/default/files/documents/usb_type-c.zip" (at 108.585 36.83 0)
+    (property "Datasheet" "https://www.usb.org/sites/default/files/documents/usb_type-c.zip" (at 104.775 13.97 0)
       (effects (font (size 1.27 1.27)) hide)
     )
@@
     )
   )
-  (symbol (lib_id "Switch:SW_Push") (at 181.61 63.5 0) (unit 1)
+  (symbol (lib_id "Switch:SW_Push") (at 181.61 63.5 0) (mirror y) (unit 1)
     (in_bom yes) (on_board yes) (dnp no)
     (property "Reference" "SW1" (at 181.61 56.261 0)
@@
       (effects (font (size 1.27 1.27)) hide)
     )
-    (pin "~")
+    (property "Part No" "" (at 255.905 102.235 0)
+      (effects (font (size 1.27 1.27)) hide)
+    )
+    (property "Note" "" (at 255.905 102.235 0)
+      (effects (font (size 1.27 1.27)) hide)
+    )
     (instances
       (project "Access"
@@
       (effects (font (size 1.27 1.27)) hide)
     )
-    (pin "~")
     (instances
       (project "Access"
@@
       (effects (font (size 1.27 1.27)) hide)
     )
-    (pin "~")
     (instances
       (project "Access"
@@
       (effects (font (size 1.27 1.27)) hide)
     )
-    (pin "~")
     (instances
       (project "Access"
@@
       (effects (font (size 1.27 1.27)) hide)
     )
-    (pin "~")
     (instances
       (project "Access"
@@
       (effects (font (size 1.27 1.27)) hide)
     )
-    (pin "~")
     (instances
       (project "Access"
@@
       (effects (font (size 1.27 1.27)) hide)
     )
-    (pin "~")
     (instances
       (project "Access"
@@
       (effects (font (size 1.27 1.27)) hide)
     )
-    (pin "~")
     (instances
       (project "Access"
@@
       (effects (font (size 1.27 1.27)) hide)
     )
-    (pin "~")
     (instances
       (project "Access"
@@
     )
   )
+  (symbol (lib_id "Diode:BAV99S") (at 151.13 97.79 0) (unit 1)
+    (in_bom yes) (on_board yes) (dnp no)
+    (property "Reference" "D1" (at 151.13 92.2782 0)
+      (effects (font (size 1.27 1.27)))
+    )
+    (property "Value" "BAV99S" (at 151.13 94.5896 0)
+      (effects (font (size 1.27 1.27)))
+    )
+    (property "Footprint" "RevK:SOT-363_SC-70-6" (at 151.13 110.49 0)
+      (effects (font (size 1.27 1.27)) hide)
+    )
+    (property "Datasheet" "https://assets.nexperia.com/documents/data-sheet/BAV99_SER.pdf" (at 151.13 97.79 0)
+      (effects (font (size 1.27 1.27)) hide)
+    )
+    (property "JLCPCB Rotation Offset" "-90" (at 151.13 97.79 0)
+      (effects (font (size 1.27 1.27)) hide)
+    )
+    (pin "1")
+    (pin "2")
+    (pin "6")
+    (pin "3")
+    (pin "4")
+    (pin "5")
+    (instances
+      (project "Access"
+        (path "/2a267270-6585-45e3-a633-b53049f10066"
+          (reference "D1") (unit 1)
+        )
+      )
+    )
+  )
   (symbol (lib_id "power:GND") (at 69.215 97.79 90) (unit 1)
     (in_bom yes) (on_board yes) (dnp no) (fields_autoplaced)
@@
       (effects (font (size 1.27 1.27)) hide)
     )
-    (pin "~")
     (instances
       (project "Access"
@@
       (effects (font (size 1.27 1.27)) hide)
     )
-    (pin "~")
     (instances
       (project "Access"
@@
       (effects (font (size 1.27 1.27)) hide)
     )
-    (pin "~")
     (instances
       (project "Access"
@@
       (effects (font (size 1.27 1.27)) hide)
     )
-    (pin "~")
+    (property "Part No" "" (at 255.905 75.565 0)
+      (effects (font (size 1.27 1.27)) hide)
+    )
+    (property "Note" "" (at 255.905 75.565 0)
+      (effects (font (size 1.27 1.27)) hide)
+    )
     (instances
       (project "Access"

Commit message: Tweak
Connections:
- net RELAY1: now also U10.6 (GPIO2); no longer U10.12 (GPIO8)
- net RELAY2: now also U10.8 (GPIO4); no longer U10.11 (GPIO7)
Changed lines of the file:
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@@
   (no_connect (at 143.51 97.79))
   (no_connect (at 38.735 102.87))
-  (no_connect (at 38.735 57.15))
+  (no_connect (at 38.735 69.85))
   (no_connect (at 151.13 102.87))
   (no_connect (at 38.735 90.17))
@@
   (no_connect (at 38.735 95.25))
   (no_connect (at 38.735 87.63))
-  (no_connect (at 38.735 54.61))
-  (no_connect (at 38.735 59.69))
+  (no_connect (at 38.735 57.15))
+  (no_connect (at 38.735 67.31))
   (no_connect (at 158.75 97.79))
   (no_connect (at 205.74 37.465))
@@
     )
   )
-  (global_label "RELAY2" (shape output) (at 38.735 67.31 180) (fields_autoplaced)
-    (effects (font (size 1.27 1.27)) (justify right))
-    (property "Intersheetrefs" "${INTERSHEET_REFS}" (at 29.6496 67.31 0)
+  (global_label "RELAY2" (shape output) (at 38.735 59.69 180) (fields_autoplaced)
+    (effects (font (size 1.27 1.27)) (justify right))
+    (property "Intersheetrefs" "${INTERSHEET_REFS}" (at 29.6496 59.69 0)
       (effects (font (size 1.27 1.27)) (justify right) hide)
     )
@@
     )
   )
-  (global_label "RELAY1" (shape output) (at 38.735 69.85 180) (fields_autoplaced)
-    (effects (font (size 1.27 1.27)) (justify right))
-    (property "Intersheetrefs" "${INTERSHEET_REFS}" (at 29.577 69.7706 0)
-      (effects (font (size 1.27 1.27)) (justify right) hide)
-    )
+  (global_label "RELAY1" (shape output) (at 38.735 54.61 180) (fields_autoplaced)
+    (effects (font (size 1.27 1.27)) (justify right))
+    (property "Intersheetrefs" "${INTERSHEET_REFS}" (at 29.577 54.5306 0)
+      (effects (font (size 1.27 1.27)) (justify right) hide)
+    )
