File: PCB/Bell/Bell.kicad_pcb (KiCad board)
At the start: 2 copper layers, 38.3 x 28.7 mm, 38 parts, among them J1 USB-C, J2 POWER, J3 Conn_01x08, J4 Shelly, J5 Conn_01x05, J6 Conn_01x02, U1 ESP32-PICO-MINI-02, U2 FT231XQ, U3 ISL89410, U4 ISL89410, U5 LMR16006XDDCR, U7 AA, U8 QR

Commit message: Library update
Parts:
- removed D2: LED_BARG, RevK:MHS190RGBCT
- removed R10: 100R, RevK:R_0603
- removed R8: 300R, RevK:R_0603
- removed R9: 1K, RevK:R_0603
- added D5: XL-1010RGBC-WS2812B, RevK:SMD1010, F.Cu at (88.7, 41.7)
Connections:
- U1 pad 33: R -> LED
- U1 pad 34: B -> unconnected-(U1-IO22-Pad34)
- U1 pad 35: G -> unconnected-(U1-IO21-Pad35)
Routing:
- net Net-(D2-Pad1): track 6.60 -> 0.00 mm
- net Net-(D2-Pad3): track 4.85 -> 0.00 mm
- net R: track 4.06 -> 0.00 mm
- net B: track 3.81 -> 0.00 mm
- net G: track 2.70 -> 0.00 mm
- net LED: track 0.00 -> 2.30 mm
- net Net-(D2-Pad4): track 1.88 -> 0.00 mm
- net +3V3: track 103.0 -> 104.4 mm
Other:
- board text added: "RGB:33"

Commit message: S3
Parts:
- removed C4: 100nF, RevK:C_0603_
- removed C5: 2.2uF, RevK:C_0805_
- removed C6: 10uF, RevK:C_0805_
- removed D4: Schottky, RevK:D_1206_
- removed J4: Shelly, RevK:Shelly
- removed L1: 6.8uH, RevK:L_4x4_
- removed R11: 100k 1%, RevK:R_0603
- removed R12: 30k 1%, RevK:R_0603
- removed U2: FT231XQ, RevK:QFN-20-1EP_4x4mm_P0.5mm_EP2.5x2.5mm
- removed U5: LMR16006XDDCR, RevK:SOT-23-Thin-6-Reg
- added C8: 1uF, RevK:C_0402, F.Cu at (90.2, 36.5)
- added C9: 100nF, RevK:C_0603_, F.Cu at (62.1, 67.2)
- added J7: Shelly, RevK:Shelly, F.Cu at (81.9, 39.6)
- added L2: 10uH, RevK:L_4x4_, F.Cu at (63.3, 70.7)
- added R8: 10K, RevK:R_0402, F.Cu at (91.2, 36.5)
- added U6: ESP32-S3-MINI-1, RevK:ESP32-S3-MINI-1, F.Cu at (81.9, 43.0)
- C1: value 0.1uF -> 10uF 50V; footprint RevK:C_0603 -> RevK:C_0603_
- C2, C3, D1: moved to F.Cu
- C7: value 10nF -> 10uF 6.3V; footprint RevK:C_0603 -> RevK:C_0603_
- R1: value 10k -> 124k; footprint RevK:R_0603 -> RevK:R_0402_
- R2: value 4k7 -> 40k2; footprint RevK:R_0603 -> RevK:R_0402_
- R3: value 10k -> 1M; footprint RevK:R_0603 -> RevK:R_0402_
- U1: value ESP32-PICO-MINI-02 -> MD8942; footprint RevK:ESP32-PICO-MINI-02 -> RevK:SOT-23-6-MD8942
- moved C1 42.8 mm to (62.1, 63.3), turned to 0 degrees
- moved R3 31.1 mm to (64.8, 67.0)
- moved R2 30.9 mm to (64.8, 65.1)
- moved AJK1 26.9 mm to (77.9, 44.5), turned to -90 degrees
- moved C7 19.3 mm to (62.1, 65.3)
- moved R1 17.9 mm to (64.8, 63.3)
- moved U1 12.2 mm to (75.8, 55.6), turned to 90 degrees
- moved D1 9.71 mm to (94.7, 39.0), turned to 0 degrees
- moved D5 9.22 mm to (94.2, 34.3)
- moved C3 7.42 mm to (97.9, 39.7), turned to -90 degrees
- moved C2 6.30 mm to (97.9, 37.1), turned to 90 degrees
- moved U8 5.30 mm to (85.3, 44.0), turned to -90 degrees
- moved D3 2.15 mm to (91.0, 48.3), turned to 90 degrees
- moved R6 1.07 mm to (89.5, 51.3)
- moved R5 0.97 mm to (85.2, 51.3)
Connections:
- U1 pad 1: GND -> unconnected-(U1-Pad1)
- U1 pad 3: +3V3 -> unconnected-(U1-Pad3)
- U1 pad 5: unconnected-(U1-I37-Pad5) -> +12V
- U1 pad 7: unconnected-(U1-I39-Pad7) -> GND
- U1 pad 8: EN -> +3V3
Routing:
- net O: track 71.0 -> 0.00 mm, vias 3 -> 0
- net +3V3: track 104.4 -> 55.9 mm, vias 6 -> 2
- net EN: track 46.3 -> 0.00 mm, vias 3 -> 0
- net I: track 40.2 -> 0.00 mm, vias 2 -> 0
- net BOOT: track 40.2 -> 0.00 mm, vias 2 -> 0
- net GND: track 29.3 -> 4.79 mm, vias 11 -> 21
- net Net-(U2-CBUS3): track 19.6 -> 0.00 mm
- net OUT3: track 23.0 -> 5.57 mm, vias 2 -> 0
- net IN1: track 28.8 -> 11.5 mm, vias 2 -> 0
- net LED: track 2.30 -> 19.1 mm, vias 0 -> 2
- net IN2: track 27.2 -> 12.1 mm, vias 2 -> 0
- net OUT1: track 21.2 -> 10.6 mm, vias 2 -> 0
- net D+: track 20.6 -> 11.0 mm
- net D-: track 21.1 -> 12.0 mm
- net Net-(J7-0): track 0.00 -> 7.47 mm
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Other:
- outline, holes or cut-outs redrawn
- board text added: "10"
- board text added: "11"
- board text added: "39"
- board text added: "40"
- board text added: "41"
- board text added: "42"
- board text added: "45"
- board text added: "46"
- board text added: "9"
- board text added: "<"
- board text added: ">"
- board text added: "Solar System Bell"
- board text added: "⎍"
- board text removed: "Solar System Bell2"

Commit message: Clean up a lot
Parts:
- C2, C3: footprint RevK:C_0603 -> RevK:C_0402
- D1: footprint Package_TO_SOT_SMD:SOT-363_SC-70-6 -> RevK:SOT-363_SC-70-6
- R4, R5, R6, R7: footprint RevK:R_0603 -> RevK:R_0402
- U3, U4: footprint Package_SO:SO-8_3.9x4.9mm_P1.27mm -> RevK:SO-8_3.9x4.9mm_P1.27mm
- moved L2 22.0 mm to (80.4, 56.9), turned to 90 degrees
- moved C9 18.8 mm to (77.8, 56.9), turned to 90 degrees
- moved C7 18.5 mm to (77.1, 54.4), turned to 180 degrees
- moved C1 15.5 mm to (77.1, 59.4), turned to 180 degrees
- moved R2 13.6 mm to (73.9, 55.1), turned to 90 degrees
- moved R3 12.3 mm to (73.9, 58.7), turned to 90 degrees
- moved R1 11.1 mm to (73.9, 56.9), turned to 90 degrees
- moved R6 6.23 mm to (92.6, 56.7), turned to 90 degrees
- moved R5 4.58 mm to (81.5, 54.0), turned to 0 degrees
- moved C2 1.36 mm to (98.3, 38.4)
- moved R4 1.32 mm to (99.3, 38.4)
- moved U1 1.30 mm to (75.8, 56.9)
- moved U6 1.10 mm to (81.8, 44.1)
- moved AJK1 1.10 mm to (77.9, 45.6)
- moved J7 1.10 mm to (81.9, 40.8)
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Routing:
- net Net-(J1-CC1): track 2.40 -> 9.06 mm, vias 0 -> 2
- net +3V3: track 55.9 -> 60.2 mm
- net Net-(J1-CC2): track 2.52 -> 5.51 mm, vias 0 -> 2
- net LED: track 19.1 -> 21.5 mm
- net OUT1: track 10.6 -> 8.23 mm
- net GND: track 4.79 -> 2.72 mm
- net D-: track 12.0 -> 9.98 mm
- net +12V: track 53.8 -> 55.2 mm
- net D+: track 11.0 -> 12.2 mm
- net T: track 1.98 -> 2.73 mm
- net GPSRX: track 11.0 -> 11.8 mm
- net GPSTICK: track 7.12 -> 6.48 mm
- net VBUS: track 17.9 -> 18.5 mm
Other:
- outline, holes or cut-outs redrawn
- board text added: "${CURRENT_DATE}"
- board text added: "+"
- board text added: "A"
- board text added: "⏚"

Commit message: LEDs
Parts:
- removed U8: QR, RevK:QR-SS
- added C10: 100nF, RevK:C_0402, F.Cu at (99.0, 39.0)
- added C11: 100nF, RevK:C_0402, F.Cu at (99.0, 44.0)
- added C12: 100nF, RevK:C_0402, F.Cu at (99.0, 47.7)
- added C13: 100nF, RevK:C_0402, F.Cu at (99.0, 50.2)
- added C4: 100nF, RevK:C_0402, F.Cu at (94.4, 33.4)
- added C5: 100nF, RevK:C_0402, F.Cu at (99.0, 32.7)
- added C6: 100nF, RevK:C_0402, F.Cu at (99.0, 35.2)
- added D10: ~, RevK:DFN1006-2L, F.Cu at (96.5, 38.1)
- added D2: XL-1010RGBC-WS2812B, RevK:SMD1010, F.Cu at (99.0, 34.0)
- added D4: XL-1010RGBC-WS2812B, RevK:SMD1010, F.Cu at (99.0, 37.7)
- added D6: XL-1010RGBC-WS2812B, RevK:SMD1010, F.Cu at (99.0, 42.7)
- added D7: XL-1010RGBC-WS2812B, RevK:SMD1010, F.Cu at (99.0, 46.5)
- added D8: XL-1010RGBC-WS2812B, RevK:SMD1010, F.Cu at (99.0, 49.0)
- added D9: XL-1010RGBC-WS2812B, RevK:SMD1010, F.Cu at (99.0, 51.5)
- D1: value BAV99S -> ~; footprint RevK:SOT-363_SC-70-6 -> RevK:DFN1006-2L
- D3: value D -> MBR0530; footprint RevK:D_1206 -> RevK:D_SOD-123
- J1: value USB-C -> USB-C-Socket-V; footprint RevK:USC16-TR -> RevK:USB-C-Socket-H
- moved D3 10.0 mm to (93.5, 38.6), turned to -90 degrees
- moved D1 5.19 mm to (96.5, 35.1), turned to 180 degrees
- moved R4 3.16 mm to (96.8, 36.4)
- moved C2 3.01 mm to (96.0, 36.4)
- moved R7 2.55 mm to (97.0, 39.3), turned to -90 degrees
- moved C3 2.37 mm to (96.2, 39.3), turned to 90 degrees
- moved U3 2.30 mm to (94.0, 49.6)
- moved U4 2.30 mm to (94.0, 44.1)
- moved D5 1.38 mm to (93.2, 33.4)
- moved AJK1 0.69 mm to (78.3, 45.1)
- turned J7 to 180 degrees
Connections:
- D1 pad 1: GND -> T
- D1 pad 2: +3V3 -> GND
- D5 pad 1: unconnected-(D5-O-Pad1) -> Net-(D2-I)
- D5 pad 2: +3V3 -> +3.3V
- D5 pad 4: LED -> RGB
- J5 pad 5: +3V3 -> +3.3V
- J7 pad 1: Net-(J7-GND) -> GND
- J7 pad 3: +3V3 -> +3.3V
- J7 pad 5: GND -> Net-(J7-Tx)
- R8 pad 1: +3V3 -> +3.3V
- U1 pad 8: +3V3 -> +3.3V
- U6 pad 3: +3V3 -> +3.3V
- U6 pad 31: LED -> OUT1
- U6 pad 32: unconnected-(U6-GPIO36-Pad32) -> OUT2
- U6 pad 35: OUT1 -> OUT3
- U6 pad 36: OUT3 -> OUT4
- U6 pad 37: OUT4 -> IN2
- U6 pad 38: OUT2 -> IN1
- U6 pad 39: Net-(J7-GND) -> Net-(J7-Tx)
- U6 pad 4: Net-(J7-Rx) -> Net-(J7-0)
- U6 pad 40: Net-(J7-0) -> Net-(J7-Rx)
- U6 pad 41: IN2 -> unconnected-(U6-GPIO45-Pad41)
- U6 pad 44: IN1 -> RGB
Routing:
- net +3.3V: track 0.00 -> 71.1 mm, vias 0 -> 1
- net +3V3: track 60.2 -> 0.00 mm, vias 2 -> 0
- net GND: track 2.72 -> 29.7 mm, vias 21 -> 19
- net LED: track 21.5 -> 0.00 mm, vias 2 -> 0
- net OUT2: track 15.1 -> 2.62 mm
- net RGB: track 0.00 -> 7.92 mm, vias 0 -> 2
- net Net-(D2-I): track 0.00 -> 6.92 mm
- net FAULT: track 2.06 -> 7.82 mm, vias 0 -> 1
- net BELL: track 2.39 -> 7.89 mm, vias 0 -> 1
- net ENGHOLD: track 2.60 -> 7.90 mm, vias 0 -> 1
- net STB: track 2.41 -> 7.68 mm, vias 0 -> 1
- net OUT1: track 8.23 -> 3.13 mm
- net +12V: track 55.2 -> 60.1 mm
- net VBUS: track 18.5 -> 22.7 mm, vias 3 -> 0
- net Net-(D4-O): track 0.00 -> 3.80 mm
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Other:
- board text added: "35"
- board text added: "36"
- board text added: "RGB:46"
- board text removed: "45"
- board text removed: "46"
- board text removed: "RGB:33"

Commit message: SMD
Parts:
- J5: footprint RevK:PTSM-HH-5-RA -> RevK:PTSM-HH-5-RA-SMD
- L2: value 10uH -> 15uH
- moved AJK1 12.8 mm to (90.8, 48.0)
- moved J5 4.34 mm to (75.5, 50.7)
- moved R5 1.41 mm to (81.7, 52.6), turned to 180 degrees
- moved R2 0.80 mm to (73.9, 54.3)
- moved R3 0.80 mm to (73.9, 57.9)
- moved C1 0.80 mm to (77.1, 58.6)
- moved C7 0.80 mm to (77.1, 53.6)
- moved C9 0.80 mm to (77.8, 56.1)
- moved L2 0.80 mm to (80.4, 56.1)
- moved R1 0.80 mm to (73.9, 56.1)
- moved U1 0.80 mm to (75.8, 56.1)
- moved J7 0.75 mm to (81.8, 40.0)
Routing:
- net +3.3V: track 71.1 -> 76.6 mm
- net GPSRX: track 12.0 -> 7.99 mm
- net GND: track 29.7 -> 33.0 mm, vias 19 -> 21
- net GPSTX: track 9.16 -> 6.79 mm
- net Net-(J1-CC1): track 8.14 -> 6.47 mm
- net D-: track 11.8 -> 13.3 mm
- net D+: track 12.1 -> 13.5 mm
- net +12V: track 60.1 -> 59.0 mm
- net IN1: track 12.6 -> 13.4 mm
- net Net-(J7-Tx): track 3.25 -> 4.01 mm
- net Net-(J7-Rx): track 6.66 -> 7.37 mm
Other:
- board size 38.3 x 28.7 mm -> 35.2 x 28.7 mm
- board text added: "GPS"

Commit message: Tweak
Parts:
- L2: value 15uH -> 10uH
Changed lines of the file:
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@@
         (effects (font (size 0.5 0.5) (thickness 0.08)))
     )
-    (fp_text value "15uH" (at 0 1.5 90) (layer "F.Fab")
+    (fp_text value "10uH" (at 0 1.5 90) (layer "F.Fab")
         (effects (font (size 0.5 0.5) (thickness 0.08)))
     )

Commit message: Cleanup
Parts:
- moved C10 1.26 mm to (99.0, 37.7)
- moved C11 1.26 mm to (99.0, 42.7)
- moved D4 1.26 mm to (99.0, 36.5)
- moved D6 1.26 mm to (99.0, 41.5)
- moved AJK1 0.57 mm to (90.5, 48.4), turned to 180 degrees
Routing:
- net Net-(D6-O): track 2.54 -> 3.80 mm
- net Net-(D2-O): track 2.56 -> 1.30 mm
Other:
- board text added: "Solar System"
- board text removed: "Solar System Bell"

Commit message: Cap
Parts:
- added C14: 100uF 6.3V, RevK:C_1206, F.Cu at (92.5, 38.8)
- moved D3 0.82 mm to (94.3, 38.8), turned to 90 degrees
- moved C2 0.60 mm to (96.7, 36.4)
- moved R4 0.60 mm to (97.5, 36.4)
- moved C3 0.54 mm to (96.7, 39.5)
- moved R7 0.54 mm to (97.5, 39.5)
Connections:
- U6 pad 33: unconnected-(U6-GPIO37-Pad33) -> GND
- U6 pad 34: unconnected-(U6-GPIO38-Pad34) -> GND
Routing:
- net GND: track 33.0 -> 20.5 mm, vias 21 -> 20
- net VBUS: track 22.7 -> 26.8 mm
- net ~{BACKLIGHT}: track 16.1 -> 20.1 mm
- net +12V: track 59.0 -> 55.0 mm
- net +3.3V: track 76.6 -> 77.9 mm
- net IN2: track 11.7 -> 12.9 mm
- net IN1: track 13.4 -> 14.6 mm
- net GPSTX: track 6.79 -> 5.79 mm
- net GPSRX: track 7.99 -> 6.99 mm
