File: PCB/Keypad/Keypad.kicad_pcb (KiCad board)
At the start: 2 copper layers, 70 x 70 mm, 26 parts, among them J1 Keypad, J2 USB-PROG, J3 Shelly, U1 SP3485, U3 ESP32-S3-MINI-1, U4 QR, U5 MD8942

Commit message: Library update
Parts:
- removed J2: USB-PROG, RevK:USB-PROG
- removed J3: Shelly, RevK:Shelly
- added J4: TC2030-USB-NL-DS, RevK:Tag-Connect_TC2030-IDC-NL_2x03_P1.27mm_Vertical, B.Cu at (104.1, 104.4)
- added REF**: Shadow, RevK:Shadow, F.Cu at (100.0, 100.0)
- moved U4 1.70 mm to (103.5, 93.8)
- moved Logo1 1.60 mm to (95.9, 94.6)
Connections:
- U3 pad 19: unconnected-(U3-GPIO15-Pad19) -> +3V3
- U3 pad 39: Net-(J3-Tx) -> unconnected-(U3-GPIO43-Pad39)
- U3 pad 4: Net-(J3-0) -> unconnected-(U3-GPIO0-Pad4)
- U3 pad 40: Net-(J3-Rx) -> unconnected-(U3-GPIO44-Pad40)
Routing:
- net D-: track 3.80 -> 16.1 mm, vias 0 -> 1
- net DC: track 24.1 -> 16.0 mm, vias 0 -> 1
- net Net-(J3-Rx): track 7.08 -> 0.00 mm
- net Net-(J3-0): track 6.67 -> 0.00 mm
- net D+: track 2.86 -> 5.87 mm, vias 0 -> 1
- net Net-(J3-Tx): track 2.94 -> 0.00 mm
- net +3V3: track 48.0 -> 47.2 mm
- net RX: track 4.60 -> 5.29 mm
- net GND: vias 19 -> 20

Commit message: Cannot make production files, FFS
Parts:
- moved C3 0.30 mm to (93.0, 107.8)
- moved J4 0.11 mm to (104.2, 104.4)
Routing:
- net GND: track 4.35 -> 8.94 mm
- net RX: track 5.29 -> 5.80 mm
Other:
- board text added: "R E"
- board text added: "R H"
- board text added: "R L"

Commit message: Render
Parts:
- removed REF**: Shadow, RevK:Shadow
Other:
- copper layers 2 -> 4
