File: PCB/Keypad/Keypad.kicad_sch (KiCad schematic)
At the start: 25 parts, among them J1 Keypad, J4 TC2030-USB-NL-DS, U1 SP3485, U3 ESP32-S3-MINI-1, U4 QR, U5 MD8942

Commit message: Tidy
Parts:
- U1: footprint RevK:SO-8_3.9x4.9mm_P1.27mm -> Package_SO:SO-8_5.3x6.2mm_P1.27mm
Connections:
- net D-: now also J4.2 (NC), J4.6 (NC)
- net DC: no longer J4.2 (VBUS)
- net GND: no longer J4.6 (GND)
Changed lines of the file:
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@@
 (kicad_sch
-	(version 20241209)
+	(version 20250114)
 	(generator "eeschema")
 	(generator_version "9.0")
@@
 			)
 		)
-		(property "Footprint" "RevK:SO-8_3.9x4.9mm_P1.27mm"
+		(property "Footprint" "Package_SO:SO-8_5.3x6.2mm_P1.27mm"
 			(at 114.3 153.67 0)
 			(effects
@@
 			)
 		)
-		(property "Description" ""
+		(property "Description" "Power symbol creates a global label with name \"+3.3V\""
 			(at 128.27 138.43 0)
 			(effects
@@
 			)
 		)
-		(property "Description" ""
+		(property "Description" "Power symbol creates a global label with name \"GND\" , ground"
 			(at 128.27 149.86 0)
 			(effects
@@
 			)
 		)
+		(property "Sim.Enable" "0"
+			(at 262.89 172.085 0)
+			(effects
+				(font
+					(size 1.27 1.27)
+				)
+				(hide yes)
+			)
+		)
 		(instances
 			(project "Faikin"
@@
 			)
 		)
-		(property "Description" ""
+		(property "Description" "Power symbol creates a global label with name \"GND\" , ground"
 			(at 90.805 107.315 0)
 			(effects
@@
 			)
 		)
-		(property "Description" ""
+		(property "Description" "Unpolarized capacitor"
 			(at 123.825 85.09 0)
 			(effects
@@
 			)
 		)
-		(property "Description" ""
+		(property "Description" "Power symbol creates a global label with name \"GND\" , ground"
 			(at 123.825 88.9 0)
 			(effects
@@
 			)
 		)
-		(property "Description" ""
+		(property "Description" "Unpolarized capacitor"
 			(at 69.215 26.035 0)
 			(effects
@@
 			)
 		)
-		(pin "~"
-		)
 		(instances
 			(project "Faikin"
@@
 			)
 		)
+		(property "Sim.Enable" "0"
+			(at 256.54 172.085 0)
+			(effects
+				(font
+					(size 1.27 1.27)
+				)
+				(hide yes)
+			)
+		)
 		(instances
 			(project "Faikin"
@@
 			)
 		)
+		(property "Sim.Enable" "0"
+			(at 259.715 175.26 0)
+			(effects
+				(font
+					(size 1.27 1.27)
+				)
+				(hide yes)
+			)
+		)
 		(instances
 			(project "Faikin"
@@
 			)
 		)
-		(property "Description" ""
+		(property "Description" "Power symbol creates a global label with name \"GND\" , ground"
 			(at 62.865 29.845 0)
 			(effects
@@
 			)
 		)
-		(pin "~"
-		)
 		(instances
 			(project "Faikin"
@@
 			)
 		)
-		(pin "~"
+		(property "Part No" ""
+			(at 187.96 60.96 0)
+			(effects
+				(font
+					(size 1.27 1.27)
+				)
+				(hide yes)
+			)
+		)
+		(property "Note" ""
+			(at 187.96 60.96 0)
+			(effects
+				(font
+					(size 1.27 1.27)
+				)
+				(hide yes)
+			)
 		)
 		(instances
@@
 	)
 	(symbol
-		(lib_name "GND_1")
 		(lib_id "power:GND")
 		(at 81.28 91.44 90)
@@
 			)
 		)
-		(property "Description" ""
+		(property "Description" "Power symbol creates a global label with name \"GND\" , ground"
 			(at 81.28 91.44 0)
 			(effects
@@
 			)
 		)
-		(pin "~"
-		)
 		(instances
 			(project "Faikin"
@@
 			)
 		)
-		(property "Description" ""
+		(property "Description" "Power symbol creates a global label with name \"+3.3V\""
 			(at 90.805 92.075 0)
 			(effects
@@
 			)
 		)
-		(property "Description" ""
+		(property "Description" "Power symbol creates a global label with name \"+3.3V\""
 			(at 155.575 55.88 0)
 			(effects
@@
 			)
 		)
-		(property "Description" ""
+		(property "Description" "Power symbol creates a global label with name \"GND\" , ground"
 			(at 167.005 65.405 0)
 			(effects
@@
 			)
 		)
+		(property "Sim.Enable" "0"
+			(at 259.715 168.91 0)
+			(effects
+				(font
+					(size 1.27 1.27)
+				)
+				(hide yes)
+			)
+		)
 		(instances
 			(project "Faikin"
@@
 			)
 		)
-		(property "Description" ""
+		(property "Description" "Power symbol creates a global label with name \"+3.3V\""
 			(at 81.28 50.8 0)
 			(effects
@@
 			)
 		)
-		(property "Description" ""
+		(property "Description" "Power symbol creates a global label with name \"+3.3V\""
 			(at 69.215 22.225 0)
 			(effects
@@
 			)
 		)
-		(property "Description" ""
+		(property "Description" "Power symbol creates a global label with name \"+3.3V\""
 			(at 123.825 81.28 0)
 			(effects
@@
 			)
 		)
-		(property "Description" ""
+		(property "Description" "Power symbol creates a global label with name \"+3.3V\""
 			(at 50.8 81.28 0)
 			(effects
@@
 			)
 		)
-		(property "Description" ""
+		(property "Description" "Power symbol creates a global label with name \"+3.3V\""
 			(at 62.865 22.225 0)
 			(effects
@@
 			)
 		)
-		(property "Description" ""
+		(property "Description" "Resistor"
 			(at 90.805 95.885 0)
 			(effects
@@
 			)
 		)
-		(property "Description" ""
+		(property "Description" "Power symbol creates a global label with name \"GND\" , ground"
 			(at 116.205 114.3 0)
 			(effects
@@
 			)
 		)
-		(pin "~"
-		)
 		(instances
 			(project "Faikin"
@@
 			)
 		)
-		(property "Description" ""
+		(property "Description" "ESP32S3"
 			(at 66.04 72.39 0)
 			(effects
@@
 			)
 		)
-		(pin "~"
-		)
 		(instances
 			(project "Faikin"
@@
 			)
 		)
-		(property "Datasheet" " ~"
+		(property "Datasheet" "~"
 			(at 123.19 56.515 0)
 			(effects
@@
 			)
 		)
-		(property "Description" ""
+		(property "Description" "Power symbol creates a global label with name \"GND\" , ground"
 			(at 69.215 29.845 0)
 			(effects
@@
 			)
 		)
-		(property "Description" ""
+		(property "Description" "Unpolarized capacitor"
 			(at 90.805 103.505 0)
 			(effects
@@
 			)
 		)
-		(property "Description" ""
+		(property "Description" "Regulator and associated components."
 			(at 167.005 55.88 0)
 			(effects
@@
 			)
 		)
-		(property "Description" ""
+		(property "Description" "Power symbol creates a global label with name \"GND\" , ground"
 			(at 114.935 88.9 0)
 			(effects
@@
 			)
 		)
-		(property "Description" ""
+		(property "Description" "Power symbol creates a global label with name \"+3.3V\""
 			(at 114.935 81.28 0)
 			(effects
@@
 			)
 		)
-		(property "Description" ""
+		(property "Description" "Generic connector, single row, 01x04, script generated (kicad-library-utils/schlib/autogen/connector/)"
 			(at 111.125 116.84 0)
 			(effects
@@
 	)
 	(symbol
-		(lib_name "GND_1")
 		(lib_id "power:GND")
 		(at 81.28 55.88 90)
@@
 			)
 		)
-		(property "Description" ""
+		(property "Description" "Power symbol creates a global label with name \"GND\" , ground"
 			(at 81.28 55.88 0)
 			(effects
@@
 			)
 		)
-		(property "Description" ""
+		(property "Description" "Unpolarized capacitor"
 			(at 62.865 26.035 0)
 			(effects
@@
 			)
 		)
-		(property "Description" ""
+		(property "Description" "RGB LED with integrated controller"
 			(at 114.935 85.09 0)
 			(effects
@@
 			)
 		)
-		(pin "~"
-		)
 		(instances
