File: PCB/Generic/Generic.kicad_sch (KiCad schematic)
At the start: 31 parts, among them J1 DC, J2 USB-C, J3 Shelly, J4 Conn_01x05, Q4 CJ2301, U1 Barcode, U2 ESP32-PICO-MINI-02, U3 CH340X, U4 MD8942, U5 QR

Commit message: VCUT
Parts:
- added V1 (x2): ~, RevK:VCUT70, symbol RevK:VCUT
Changed lines of the file:
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@@
+    )
+  )
+  (symbol (lib_id "RevK:VCUT") (at 262.89 171.45 0) (unit 1)
+    (in_bom yes) (on_board yes) (dnp no) (fields_autoplaced)
+    (property "Reference" "V1" (at 262.89 170.18 0)
+      (effects (font (size 1.27 1.27)) hide)
+    )
+    (property "Value" "~" (at 262.89 171.45 0)
+      (effects (font (size 1.27 1.27)))
+    )
+    (property "Footprint" "RevK:VCUT70" (at 262.89 172.72 0)
+      (effects (font (size 1.27 1.27)) hide)
+    )
+    (property "Datasheet" "" (at 262.89 171.45 0)
+      (effects (font (size 1.27 1.27)) hide)
+    )
+    (instances
+      (project "Reference"
+        (path "/825c70b0-4860-42b7-97dc-86bfa46e06fd"
+          (reference "V1") (unit 1)
+        )
+      )
+      (project "Generic"
+        (path "/babeabf2-f3b0-4ed5-8d9e-0215947e6cf3"
+          (reference "V2") (unit 1)
+        )
+      )
     )
   )
@@
         )
       )
+    )
+  )
+  (symbol (lib_id "RevK:VCUT") (at 262.89 177.8 0) (unit 1)
+    (in_bom yes) (on_board yes) (dnp no) (fields_autoplaced)
+    (property "Reference" "V1" (at 262.89 176.53 0)
+      (effects (font (size 1.27 1.27)) hide)
+    )
+    (property "Value" "~" (at 262.89 177.8 0)
+      (effects (font (size 1.27 1.27)))
+    )
+    (property "Footprint" "RevK:VCUT70" (at 262.89 179.07 0)
+      (effects (font (size 1.27 1.27)) hide)
+    )
+    (property "Datasheet" "" (at 262.89 177.8 0)
+      (effects (font (size 1.27 1.27)) hide)
+    )
+    (instances
+      (project "Reference"
+        (path "/825c70b0-4860-42b7-97dc-86bfa46e06fd"
+          (reference "V1") (unit 1)
+        )
+      )
+      (project "Generic"
+        (path "/babeabf2-f3b0-4ed5-8d9e-0215947e6cf3"
+          (reference "V1") (unit 1)
+        )
+      )

Commit message: CH340X DTR
Parts:
- removed R6: 4k7, RevK:R_0402, symbol Device:R
- V1: now left out of the parts list
Connections:
- net BOOT: now also U3.5 (~{CTS})
Changed lines of the file:
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@@
   (junction (at 184.785 36.83) (diameter 0) (color 0 0 0 0)
   )
+  (junction (at 175.895 112.395) (diameter 0) (color 0 0 0 0)
+  )
   (junction (at 81.28 57.15) (diameter 0) (color 0 0 0 0)
   )
@@
   )
   (junction (at 159.385 68.58) (diameter 0) (color 0 0 0 0)
-  )
-  (junction (at 177.8 112.395) (diameter 0) (color 0 0 0 0)
   )
   (junction (at 165.735 90.805) (diameter 0) (color 0 0 0 0)
@@
     (stroke (width 0) (type default))
   )
-  (wire (pts (xy 175.895 104.775) (xy 177.8 104.775))
-    (stroke (width 0) (type default))
-  )
-  (wire (pts (xy 175.895 112.395) (xy 177.8 112.395))
-    (stroke (width 0) (type default))
-  )
   (wire (pts (xy 47.625 48.26) (xy 50.8 48.26))
     (stroke (width 0) (type default))
   )
-  (wire (pts (xy 177.8 112.395) (xy 180.34 112.395))
+  (wire (pts (xy 175.895 112.395) (xy 180.34 112.395))
     (stroke (width 0) (type default))
   )
@@
   )
   (wire (pts (xy 57.785 160.02) (xy 69.85 160.02))
+    (stroke (width 0) (type default))
+  )
+  (wire (pts (xy 175.895 104.775) (xy 175.895 112.395))
     (stroke (width 0) (type default))
   )
@@
     )
   )
-  (global_label "BOOT" (shape output) (at 180.34 112.395 0) (fields_autoplaced)
-    (effects (font (size 1.27 1.27)) (justify left))
-    (property "Intersheetrefs" "${INTERSHEET_REFS}" (at 187.4902 112.395 0)
+  (global_label "BOOT" (shape output) (at 177.165 112.395 0) (fields_autoplaced)
+    (effects (font (size 1.27 1.27)) (justify left))
+    (property "Intersheetrefs" "${INTERSHEET_REFS}" (at 184.3152 112.395 0)
       (effects (font (size 1.27 1.27)) (justify left) hide)
     )
@@
         (path "/babeabf2-f3b0-4ed5-8d9e-0215947e6cf3"
           (reference "D4") (unit 2)
-        )
-      )
-    )
-  )
-  (symbol (lib_id "Device:R") (at 177.8 108.585 0) (unit 1)
-    (in_bom yes) (on_board yes) (dnp no)
-    (property "Reference" "R6" (at 179.705 108.585 90)
-      (effects (font (size 1.27 1.27)))
-    )
-    (property "Value" "4k7" (at 177.8 108.585 90)
-      (effects (font (size 1.27 1.27)))
-    )
-    (property "Footprint" "RevK:R_0402" (at 176.022 108.585 90)
-      (effects (font (size 1.27 1.27)) hide)
-    )
-    (property "Datasheet" "~" (at 177.8 108.585 0)
-      (effects (font (size 1.27 1.27)) hide)
-    )
-    (pin "1")
-    (pin "2")
-    (instances
-      (project "Generic"
-        (path "/babeabf2-f3b0-4ed5-8d9e-0215947e6cf3"
-          (reference "R6") (unit 1)
         )
       )
@@
   )
   (symbol (lib_id "RevK:VCUT") (at 262.89 171.45 0) (unit 1)
-    (in_bom yes) (on_board yes) (dnp no) (fields_autoplaced)
+    (in_bom no) (on_board yes) (dnp no) (fields_autoplaced)
     (property "Reference" "V1" (at 262.89 170.18 0)
       (effects (font (size 1.27 1.27)) hide)
@@
     )
     (property "Datasheet" "" (at 262.89 171.45 0)
+      (effects (font (size 1.27 1.27)) hide)
+    )
+    (property "Sim.Enable" "0" (at 262.89 171.45 0)
       (effects (font (size 1.27 1.27)) hide)
     )
@@
   )
   (symbol (lib_id "RevK:VCUT") (at 262.89 177.8 0) (unit 1)
-    (in_bom yes) (on_board yes) (dnp no) (fields_autoplaced)
+    (in_bom no) (on_board yes) (dnp no) (fields_autoplaced)
     (property "Reference" "V1" (at 262.89 176.53 0)
       (effects (font (size 1.27 1.27)) hide)
@@
       (effects (font (size 1.27 1.27)) hide)
     )
+    (property "Sim.Enable" "0" (at 262.89 177.8 0)
+      (effects (font (size 1.27 1.27)) hide)
+    )

Commit message: Fix RGB
Parts:
- D1: symbol Device:LED_RBGA -> Device:LED_RGBA
Connections:
- net at R2.1: now also D1.2 (GK); no longer D1.3 (GK)
- net at R3.1: now also D1.3 (BK); no longer D1.2 (BK)
Changed lines of the file:
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@@
     )
   )
-  (symbol (lib_id "Device:LED_RBGA") (at 169.545 153.67 0) (unit 1)
+  (symbol (lib_id "Device:LED_RGBA") (at 169.545 153.67 0) (unit 1)
     (in_bom yes) (on_board yes) (dnp no)
     (property "Reference" "D1" (at 169.545 141.0462 0)

Commit message: Some improvement, needs to change to S3 though
Parts:
- removed D1: RGB, RevK:LED-RGB-1.6x1.6, symbol Device:LED_RGBA
- removed R1: 680R, RevK:R_0402, symbol Device:R
- removed R2: 2K, RevK:R_0402, symbol Device:R
- removed R3: 220R, RevK:R_0402, symbol Device:R
- removed U1: Barcode, RevK:EAN-5060634238113, symbol RevK:Barcode
- added D4: XL-1010RGBC-WS2812B, RevK:SMD1010, symbol RevK:WS2812B-1mm
Connections:
- net +3.3V: now also D4.2 (+)
- net GND: now also D4.3 (-)
- net B: no longer names the net of U2.35 (IO21)
- net G renamed LED
- net LED: now also D4.4 (I)
- net R: no longer names the net of U2.34 (IO22)
- no-connect marks 20 -> 23

Commit message: S3
Parts:
- removed J3: Shelly, RevK:Shelly, symbol RevK:Shelly
- removed R1: 10k, RevK:R_0402, symbol Device:R
- removed U2: ESP32-PICO-MINI-02, RevK:ESP32-PICO-MINI-02, symbol RevK:ESP32-PICO-MINI-02
- removed U3: CH340X, RevK:CH340X, symbol RevK:CH340X
- added C20: 1uF, RevK:C_0402, symbol Device:C
- added J8: Shelly, RevK:Shelly, symbol RevK:Shelly
- added R26: 10K, RevK:R_0402, symbol Device:R
- added U10: ESP32-S3-MINI-1, RevK:ESP32-S3-MINI-1, symbol RevK:ESP32-S3-MINI-1-N4R2
- C1: value 0.1uF -> 100nF
Connections:
- net +3.3V: now also J8.3 (3V3), R26.1, U10.3 (3V3)
- net D+: now also U10.24 (GPIO20)
- net D-: now also U10.23 (GPIO19)
- net GND: now also C20.2, J8.1 (GND), U10.1 (GND), U10.17 (GPIO13), U10.18 (GPIO14), U10.19 (GPIO15), U10.2 (GND), U10.20 (GPIO16), U10.21 (GPIO17), U10.22 (GPIO18), U10.25 (GPIO21), U10.42 (GND), U10.43 (GND), U10.46 (GND), U10.47 (GND), U10.48 (GND), U10.49 (GND), U10.50 (GND), U10.51 (GND), U10.52 (GND), U10.53 (GND), U10.54 (GND), U10.55 (GND), U10.56 (GND), U10.57 (GND), U10.58 (GND), U10.59 (GND), U10.60 (GND), U10.61 (GND), U10.62 (GND), U10.63 (GND), U10.64 (GND), U10.65 (GND)
- net GPSRX: now also U10.29 (GPIO34)
- net GPSTX: now also U10.30 (GPIO48)
- net LED: now also U10.16 (GPIO12)
- net TICK: now also U10.31 (GPIO35)
- new net: C20.1, R26.2, U10.45 (EN)
- new net: J8.2 (0), U10.4 (GPIO0)
- new net: J8.4 (Rx), U10.40 (GPIO44)
- new net: J8.5 (Tx), U10.39 (GPIO43)
- no-connect marks 23 -> 25
Other:
- moved on the sheet: C1

Commit message: Library update
Parts:
- C5: value 10uF 50V -> 10uF 35V; LCSC Part # C1591 -> C194427
Changed lines of the file:
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@@
       (effects (font (size 1.27 1.27)) (justify left))
     )
-    (property "Value" "10uF 50V" (at 256.54 29.845 0)
+    (property "Value" "10uF 35V" (at 256.54 29.845 0)
       (effects (font (size 1.27 1.27)) (justify left))
     )
@@
       (effects (font (size 1.27 1.27)) hide)
     )
-    (property "LCSC Part #" "C1591" (at 250.19 29.845 0)
+    (property "LCSC Part #" "C194427" (at 250.19 29.845 0)
       (effects (font (size 1.27 1.27)) hide)
     )

Commit message: Tidy
Parts:
- renumbered C20 to C2, D4 to D2, D2 to D4, D2 to D5, J8 to J5, Q4 to Q1, R26 to R4, U10 to U1, V1 to V2

Commit message: PCB Update
Parts:
- removed U5: QR, RevK:QR-SS, symbol RevK:QR
- C5: LCSC Part # C194427 -> (none); MPN (none) -> C194427
- C6: LCSC Part # C1691 -> (none); MPN (none) -> C1691
- D1: LCSC Part # C143805 -> (none); MPN (none) -> C143805
- D2: LCSC Part # C5349953 -> (none); MPN (none) -> C5349953
- D4, D5: JLCPCB Rotation Offset 90 -> (none)
- J2: value USB-C -> USB-C-Socket-V; footprint RevK:USC16-TR -> RevK:USB-C-Socket-H; symbol RevK:USB-C -> RevK:USB-C-Socket-H; JLCPCB Rotation Offset 0 -> (none); LCSC Part # C709357 -> (none); MPN (none) -> C709357
- Q1: JLCPCB Rotation Offset 180 -> (none); LCSC Part  C2910170 -> (none); MPN (none) -> C2910170
- U1: LCSC Part # C3013941 -> (none); MPN (none) -> C3013941
- U4: LCSC Part # C2684786 -> (none); MPN (none) -> C2684786
Changed lines of the file:
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@@
 	)
 	(symbol
-		(lib_id "RevK:USB-C")
+		(lib_id "RevK:USB-C-Socket-H")
 		(at 159.385 45.72 0)
 		(unit 1)
@@
 		(dnp no)
 		(property "Reference" "J2"
-			(at 162.1028 23.6982 0)
+			(at 149.225 26.67 0)
 			(effects
 				(font
 					(size 1.27 1.27)
 				)
+				(justify left)
 			)
 		)
-		(property "Value" "USB-C"
-			(at 162.1028 26.0096 0)
+		(property "Value" "USB-C-Socket-V"
+			(at 160.02 33.02 0)
 			(effects
 				(font
@@
 			)
 		)
-		(property "Footprint" "RevK:USC16-TR"
+		(property "Footprint" "RevK:USB-C-Socket-H"
 			(at 159.385 25.4 0)
 			(effects
@@
 			)
 		)
-		(property "Description" ""
-			(at 159.385 45.72 0)
-			(effects
-				(font
-					(size 1.27 1.27)
-				)
-			)
-		)
-		(property "LCSC Part #" "C709357"
+		(property "Description" "USB 2.0-only Type-C Receptacle connector"
 			(at 159.385 45.72 0)
 			(effects
@@
 			)
 		)
-		(property "JLCPCB Rotation Offset" "0"
+		(property "MPN" "C709357"
 			(at 159.385 45.72 0)
 			(effects
@@
 			)
 		)
-		(property "LCSC Part #" "C143805"
+		(property "MPN" "C143805"
 			(at 193.675 30.48 0)
 			(effects
@@
 			)
 		)
-		(property "JLCPCB Rotation Offset" "90"
-			(at 57.785 128.905 0)
-			(effects
-				(font
-					(size 1.27 1.27)
-				)
-				(hide yes)
-			)
-		)
 		(pin "1"
 		)
@@
 			)
 		)
-		(property "LCSC Part " "C2910170"
-			(at 74.93 162.56 90)
-			(effects
-				(font
-					(size 1.27 1.27)
-				)
-				(hide yes)
-			)
-		)
-		(property "JLCPCB Rotation Offset" "180"
+		(property "MPN" "C2910170"
 			(at 74.93 162.56 90)
 			(effects
@@
 			)
 		)
-		(property "JLCPCB Rotation Offset" "90"
-			(at 98.425 128.905 0)
-			(effects
-				(font
-					(size 1.27 1.27)
-				)
-				(hide yes)
-			)
-		)
 		(pin "1"
 		)
@@
 			)
 		)
-		(property "LCSC Part #" "C1691"
+		(property "MPN" "C1691"
 			(at 250.19 31.75 0)
 			(effects
@@
 			)
 		)
-		(property "JLCPCB Rotation Offset" "90"
-			(at 36.83 128.905 0)
-			(effects
-				(font
-					(size 1.27 1.27)
-				)
-				(hide yes)
-			)
-		)
 		(pin "1"
 		)
@@
 			)
 		)
-		(property "LCSC Part #" "C5349953"
+		(property "MPN" "C5349953"
 			(at 203.2 94.615 0)
 			(effects
@@
 			)
 		)
-		(property "LCSC Part #" "C2684786"
+		(property "MPN" "C2684786"
 			(at 229.235 62.865 0)
 			(effects
@@
 			)
 		)
-		(property "LCSC Part #" "C3013941"
+		(property "MPN" "C3013941"
 			(at 53.975 93.98 0)
 			(effects
@@
 	)
 	(symbol
-		(lib_id "RevK:QR")
-		(at 271.78 173.99 0)
-		(unit 1)
-		(exclude_from_sim no)
-		(in_bom no)
-		(on_board yes)
-		(dnp no)
-		(fields_autoplaced yes)
-		(property "Reference" "U5"
-			(at 271.78 177.165 0)
-			(effects
-				(font
-					(size 1.27 1.27)
-				)
-				(hide yes)
-			)
-		)
-		(property "Value" "QR"
-			(at 271.78 177.165 0)
-			(effects
-				(font
-					(size 1.27 1.27)
-				)
-				(hide yes)
-			)
-		)
-		(property "Footprint" "RevK:QR-SS"
-			(at 271.145 174.625 0)
-			(effects
-				(font
-					(size 1.27 1.27)
-				)
-				(hide yes)
-			)
-		)
-		(property "Datasheet" ""
-			(at 271.145 174.625 0)
-			(effects
-				(font
-					(size 1.27 1.27)
-				)
-				(hide yes)
-			)
-		)
-		(property "Description" ""
-			(at 271.78 173.99 0)
-			(effects
-				(font
-					(size 1.27 1.27)
-				)
-			)
-		)
-		(property "Note" "Non part, PCB printed"
-			(at 271.78 173.99 0)
-			(effects
-				(font
-					(size 1.27 1.27)
-				)
-				(hide yes)
-			)
-		)
-		(instances
-			(project "Generic"
-				(path "/babeabf2-f3b0-4ed5-8d9e-0215947e6cf3"
-					(reference "U5")
-					(unit 1)
-				)
-			)
-		)
-	)
-	(symbol
 		(lib_id "RevK:VCUT")
 		(at 262.89 177.8 0)
@@
 			)
 		)
-		(property "LCSC Part #" "C194427"
+		(property "MPN" "C194427"
 			(at 250.19 29.845 0)
 			(effects
@@
 			)
 		)
-		(property "JLCPCB Rotation Offset" "90"
-			(at 78.74 128.905 0)
-			(effects
-				(font
-					(size 1.27 1.27)
-				)
-				(hide yes)
-			)
-		)
